File: Fancy-7-Segment-LED-Clock.sch (KiCad schematic (older format))
At the start: 66 parts, among them J1 Conn_02x04_Odd_Even, J2 Conn_02x04_Odd_Even, J3 Conn_02x04_Odd_Even, J4 Conn_02x04_Odd_Even, U1 TLC5952, U2 TLC5952

Commit message: ...
Parts:
- D1, D10, D11, D12, D13, D14, D15, D16, D17, D18, D19, D2, D20, D21, D22, D23, D24, D25, D26, D27, D28, D29, D3, D30, D31, D32, D33, D34, D35, D36, D37, D38, D39, D4, D40, D41, D42, D43, D44, D45, D46, D47, D48, D49, D5, D50, D51, D52, D53, D54, D55, D56, D6, D7, D8, D9: footprint ak:CREE_PLCC6_5.5x5.5 -> LED_SMD:LED_RGB_5050-6
- J1, J3: footprint ak:TE_5147722-3 -> ak:HARWIN_M20-8890845
- J2, J4: footprint (none) -> ak:HARWIN_M20-7910842R

Commit message: ...
Parts:
- added R10, R11, R12, R13, R14, R15, R16, R3, R4, R5, R6, R7, R8, R9: R_Small, Resistors_SMD:R_0805, symbol Device:R_Small
Connections:
- net at D1.3 (RK): now also R3.1; no longer U1.5 (OUTR0)
- net at D9.3 (RK): now also R4.1; no longer U1.8 (OUTR1)
- net at D17.3 (RK): now also R5.1; no longer U1.11 (OUTR2)
- net at D25.3 (RK): now also R6.1; no longer U1.14 (OUTR3)
- net at D33.3 (RK): now also R7.1; no longer U1.17 (OUTR4)
- net at D41.3 (RK): now also R8.1; no longer U1.20 (OUTR5)
- net at D49.3 (RK): now also R9.1; no longer U1.23 (OUTR6)
- net at D53.3 (RK): now also R10.1; no longer U1.26 (OUTR7)
- net at D45.3 (RK): now also R16.1; no longer U2.26 (OUTR7)
- net at D37.3 (RK): now also R15.1; no longer U2.23 (OUTR6)
- net at D21.3 (RK): now also R13.1; no longer U2.17 (OUTR4)
- net at D13.1 (BK): now also R12.1; no longer U2.16 (OUTB3)
- net at D5.3 (RK): now also R11.1; no longer U2.11 (OUTR2)
- net at D29.3 (RK): now also R14.1; no longer U2.20 (OUTR5)
- new net: R3.2, U1.5 (OUTR0)
- new net: R4.2, U1.8 (OUTR1)
- new net: R5.2, U1.11 (OUTR2)
- new net: R6.2, U1.14 (OUTR3)
- new net: R7.2, U1.17 (OUTR4)
- new net: R8.2, U1.20 (OUTR5)
- new net: R9.2, U1.23 (OUTR6)
- new net: R10.2, U1.26 (OUTR7)
- new net: R12.2, U2.16 (OUTB3)
- new net: R13.2, U2.17 (OUTR4)
- new net: R14.2, U2.20 (OUTR5)
- new net: R15.2, U2.23 (OUTR6)
- new net: R16.2, U2.26 (OUTR7)
- new net: R11.2, U2.11 (OUTR2)
Changed lines of the file:
@@
 	5100 3850 5950 3850
 Wire Wire Line
-	5000 3650 5950 3650
+	5000 3650 5650 3650
 Wire Wire Line
 	4850 3200 5950 3200
@@
 	4750 3000 5950 3000
 Wire Wire Line
-	4650 2800 5950 2800
+	4650 2800 5650 2800
 Wire Wire Line
 	4450 2350 5950 2350
@@
 	4350 2150 5950 2150
 Wire Wire Line
-	4250 1950 5950 1950
+	4250 1950 5650 1950
 $Comp
 L ak:LED_BGR D1
@@
 $EndComp
 Wire Wire Line
-	5600 5400 5950 5400
+	5600 5400 5650 5400
 Wire Wire Line
 	5500 5600 5950 5600
@@
 	5400 5800 5950 5800
 Wire Wire Line
-	5250 6250 5950 6250
+	5250 6250 5650 6250
 Wire Wire Line
 	5150 6450 5950 6450
@@
 	5050 6650 5950 6650
 Wire Wire Line
-	4850 7100 5950 7100
+	4850 7100 5650 7100
 Wire Wire Line
 	4750 7300 5950 7300
@@
 Connection ~ 7750 7500
 Wire Wire Line
-	4450 7950 5950 7950
+	4450 7950 5650 7950
 Wire Wire Line
 	4350 8150 5950 8150
@@
 	5400 4850 5400 4500
 Wire Wire Line
-	5400 4500 5950 4500
+	5400 4500 5650 4500
 Wire Wire Line
 	4150 4950 5500 4950
@@
 	11500 3850 12350 3850
 Wire Wire Line
-	11400 3650 12350 3650
-Wire Wire Line
-	12000 5400 12350 5400
+	11400 3650 12100 3650
+Wire Wire Line
+	12000 5400 12100 5400
 Wire Wire Line
 	11900 5600 12350 5600
@@
 	11800 5800 12350 5800
 Wire Wire Line
-	11650 6250 12350 6250
+	11650 6250 12100 6250
 Wire Wire Line
 	11550 6450 12350 6450
@@
 	11450 6650 12350 6650
 Wire Wire Line
-	11250 7100 12350 7100
+	11250 7100 12100 7100
 Wire Wire Line
 	11150 7300 12350 7300
@@
 	11050 7500 12350 7500
 Wire Wire Line
-	10850 7950 12350 7950
+	10850 7950 12100 7950
 Wire Wire Line
 	10750 8150 12350 8150
@@
 	12000 5050 12000 4900
 Wire Wire Line
-	12000 4900 12350 4900
+	12000 4900 12100 4900
 Connection ~ 14150 3650
 Wire Wire Line
@@
 	1    0    0    -1
 $EndComp
+$Comp
+L Device:R_Small R3
+U 1 1 5D748E11
+P 5750 1950
+F 0 "R3" V 5554 1950 50  0000 C CNN
+F 1 "R_Small" V 5645 1950 50  0000 C CNN
+F 2 "Resistors_SMD:R_0805" H 5750 1950 50  0001 C CNN
+F 3 "~" H 5750 1950 50  0001 C CNN
+	1    5750 1950
+	0    1    1    0
+$EndComp
+Wire Wire Line
+	5850 1950 5950 1950
+$Comp
+L Device:R_Small R4
+U 1 1 5D749A2B
+P 5750 2800
+F 0 "R4" V 5554 2800 50  0000 C CNN
+F 1 "R_Small" V 5645 2800 50  0000 C CNN
+F 2 "Resistors_SMD:R_0805" H 5750 2800 50  0001 C CNN
+F 3 "~" H 5750 2800 50  0001 C CNN
+	1    5750 2800
+	0    1    1    0
+$EndComp
+Wire Wire Line
+	5850 2800 5950 2800
+$Comp
+L Device:R_Small R5
+U 1 1 5D749F3B
+P 5750 3650
+F 0 "R5" V 5554 3650 50  0000 C CNN
+F 1 "R_Small" V 5645 3650 50  0000 C CNN
+F 2 "Resistors_SMD:R_0805" H 5750 3650 50  0001 C CNN
+F 3 "~" H 5750 3650 50  0001 C CNN
+	1    5750 3650
+	0    1    1    0
+$EndComp
+Wire Wire Line
+	5850 3650 5950 3650
+$Comp
+L Device:R_Small R6
+U 1 1 5D74A5E4
+P 5750 4500
+F 0 "R6" V 5554 4500 50  0000 C CNN
+F 1 "R_Small" V 5645 4500 50  0000 C CNN
+F 2 "Resistors_SMD:R_0805" H 5750 4500 50  0001 C CNN
+F 3 "~" H 5750 4500 50  0001 C CNN
+	1    5750 4500
+	0    1    1    0
+$EndComp
+Wire Wire Line
+	5850 4500 5950 4500
+$Comp
+L Device:R_Small R7
+U 1 1 5D74AB76
+P 5750 5400
+F 0 "R7" V 5554 5400 50  0000 C CNN
+F 1 "R_Small" V 5645 5400 50  0000 C CNN
+F 2 "Resistors_SMD:R_0805" H 5750 5400 50  0001 C CNN
+F 3 "~" H 5750 5400 50  0001 C CNN
+	1    5750 5400
+	0    1    1    0
+$EndComp
+Wire Wire Line
+	5850 5400 5950 5400
+$Comp
+L Device:R_Small R8
+U 1 1 5D7EDBCE
+P 5750 6250
+F 0 "R8" V 5554 6250 50  0000 C CNN
+F 1 "R_Small" V 5645 6250 50  0000 C CNN
+F 2 "Resistors_SMD:R_0805" H 5750 6250 50  0001 C CNN
+F 3 "~" H 5750 6250 50  0001 C CNN
+	1    5750 6250
+	0    1    1    0
+$EndComp
+Wire Wire Line
+	5850 6250 5950 6250
+$Comp
+L Device:R_Small R9
+U 1 1 5D7EE07E
+P 5750 7100
+F 0 "R9" V 5554 7100 50  0000 C CNN
+F 1 "R_Small" V 5645 7100 50  0000 C CNN
+F 2 "Resistors_SMD:R_0805" H 5750 7100 50  0001 C CNN
+F 3 "~" H 5750 7100 50  0001 C CNN
+	1    5750 7100
+	0    1    1    0
+$EndComp
+Wire Wire Line
+	5850 7100 5950 7100
+$Comp
+L Device:R_Small R10
+U 1 1 5D7EE3E2
+P 5750 7950
+F 0 "R10" V 5554 7950 50  0000 C CNN
+F 1 "R_Small" V 5645 7950 50  0000 C CNN
+F 2 "Resistors_SMD:R_0805" H 5750 7950 50  0001 C CNN
+F 3 "~" H 5750 7950 50  0001 C CNN
+	1    5750 7950
+	0    1    1    0
+$EndComp
+Wire Wire Line
+	5850 7950 5950 7950
+$Comp
+L Device:R_Small R12
+U 1 1 5D7EE7C3
+P 12200 4900
+F 0 "R12" V 12004 4900 50  0000 C CNN
+F 1 "R_Small" V 12095 4900 50  0000 C CNN
+F 2 "Resistors_SMD:R_0805" H 12200 4900 50  0001 C CNN
+F 3 "~" H 12200 4900 50  0001 C CNN
+	1    12200 4900
+	0    1    1    0
+$EndComp
+Wire Wire Line
+	12300 4900 12350 4900
+$Comp
+L Device:R_Small R13
+U 1 1 5D7EF6A4
+P 12200 5400
+F 0 "R13" V 12004 5400 50  0000 C CNN
+F 1 "R_Small" V 12095 5400 50  0000 C CNN
+F 2 "Resistors_SMD:R_0805" H 12200 5400 50  0001 C CNN
+F 3 "~" H 12200 5400 50  0001 C CNN
+	1    12200 5400
+	0    1    1    0
+$EndComp
+Wire Wire Line
+	12300 5400 12350 5400
+$Comp
+L Device:R_Small R14
+U 1 1 5D7EFA0D
+P 12200 6250
+F 0 "R14" V 12004 6250 50  0000 C CNN
+F 1 "R_Small" V 12095 6250 50  0000 C CNN
+F 2 "Resistors_SMD:R_0805" H 12200 6250 50  0001 C CNN
+F 3 "~" H 12200 6250 50  0001 C CNN
+	1    12200 6250
+	0    1    1    0
+$EndComp
+Wire Wire Line
+	12300 6250 12350 6250
+$Comp
+L Device:R_Small R15
+U 1 1 5D7EFDDA
+P 12200 7100
+F 0 "R15" V 12004 7100 50  0000 C CNN
+F 1 "R_Small" V 12095 7100 50  0000 C CNN
+F 2 "Resistors_SMD:R_0805" H 12200 7100 50  0001 C CNN
+F 3 "~" H 12200 7100 50  0001 C CNN
+	1    12200 7100
+	0    1    1    0
+$EndComp
+Wire Wire Line
+	12300 7100 12350 7100
+$Comp
+L Device:R_Small R16
+U 1 1 5D7F048B
+P 12200 7950
+F 0 "R16" V 12004 7950 50  0000 C CNN
+F 1 "R_Small" V 12095 7950 50  0000 C CNN
+F 2 "Resistors_SMD:R_0805" H 12200 7950 50  0001 C CNN
+F 3 "~" H 12200 7950 50  0001 C CNN
+	1    12200 7950
+	0    1    1    0
+$EndComp
+Wire Wire Line
+	12300 7950 12350 7950
+$Comp
+L Device:R_Small R11
+U 1 1 5D7F0927
+P 12200 3650
+F 0 "R11" V 12004 3650 50  0000 C CNN
+F 1 "R_Small" V 12095 3650 50  0000 C CNN
+F 2 "Resistors_SMD:R_0805" H 12200 3650 50  0001 C CNN
+F 3 "~" H 12200 3650 50  0001 C CNN
+	1    12200 3650
+	0    1    1    0
+$EndComp
+Wire Wire Line
+	12300 3650 12350 3650
 $EndSCHEMATC
