File: Fancy-7-Segment-LED-Clock.sch (KiCad schematic (older format))
At the start: 80 parts, among them J1 Conn_02x04_Odd_Even, J2 Conn_02x04_Odd_Even, J3 Conn_02x04_Odd_Even, J4 Conn_02x04_Odd_Even, U1 TLC5952, U2 TLC5952

Commit message: all change...
Parts:
- J1, J2: value Conn_02x04_Odd_Even -> Conn_02x04_Top_Bottom; symbol Connector_Generic:Conn_02x04_Odd_Even -> Connector_Generic:Conn_02x04_Top_Bottom
Connections:
- net GND: now also J1.4 (Pin_4), J1.6 (Pin_6), J2.4 (Pin_4), J2.6 (Pin_6); no longer J1.1 (Pin_1), J1.7 (Pin_7), J2.1 (Pin_1), J2.7 (Pin_7)
- net VCC: now also J1.7 (Pin_7), J2.7 (Pin_7); no longer J1.6 (Pin_6), J2.6 (Pin_6)
- net Vdrive: now also J1.1 (Pin_1), J2.1 (Pin_1); no longer J1.4 (Pin_4), J2.4 (Pin_4)
Other:
- moved on the sheet: J2

Commit message: Added line driver. Routing.
Parts:
- added C10, C11, C7, C8, C9: 100n, Capacitor_SMD:C_0805_2012Metric, symbol Device:C_Small
- added C3, C4, C5, C6: 47uF, Capacitor_SMD:C_Elec_6.3x5.8, symbol Device:CP_Small
- added D57, D62: D_TVS, Diode_SMD:D_SMA, symbol Device:D_TVS
- added D58, D59, D60, D61: 5V, Diode_SMD:D_SOD-323, symbol Device:D_TVS
- added JP1, JP2, JP3, JP4: SolderJumper_2_Open, Jumper:SolderJumper-2_P1.3mm_Open_TrianglePad1.0x1.5mm, symbol Jumper:SolderJumper_2_Open
- added U3: 74LS244, Package_SO:SO-20_12.8x7.5mm_P1.27mm, symbol 74xx:74LS244
- C1, C2: value C_Small -> 100n
- J1: value Conn_02x04_Top_Bottom -> Power In
- J2: value Conn_02x04_Top_Bottom -> Power out
- J3: value Conn_02x04_Odd_Even -> Signal in
- J4: value Conn_02x04_Odd_Even -> Signal out
Connections:
- net BLANK: now also JP4.1 (A), U3.3 (O3b); no longer J3.8 (Pin_8), J4.8 (Pin_8)
- net GND: now also U1.33 (EPAD), U2.33 (EPAD), C10.2, C11.2, C3.2, C4.2, C5.2, C6.2, C7.2, C8.2, C9.2, D57.2 (A2), D58.2 (A2), D59.2 (A2), D60.2 (A2), D61.2 (A2), D62.2 (A2), U3.10 (GND), U3.19 (OEb), U3.2 (I0a), U3.4 (I1a), U3.6 (I2a), U3.8 (I3a)
- net LAT: now also JP3.1 (A), U3.5 (O2b); no longer J3.2 (Pin_2), J4.2 (Pin_2)
- net SCLK: now also JP2.1 (A), U3.7 (O1b); no longer J3.4 (Pin_4), J4.4 (Pin_4)
- net SIN: now also U3.9 (O0b); no longer J3.6 (Pin_6)
- net SOUT: now also JP1.1 (A); no longer J4.6 (Pin_6)
- net VCC: now also C10.1, C3.1, C5.1, C7.1, C8.1, D57.1 (A1), U3.1 (OEa), U3.20 (VCC)
- net Vdrive: now also C11.1, C4.1, C6.1, C9.1, D62.1 (A1)
- new net: D58.1 (A1), J3.2 (Pin_2), U3.11 (I0b)
- new net: D59.1 (A1), J3.4 (Pin_4), U3.13 (I1b)
- new net: D60.1 (A1), J3.6 (Pin_6), U3.15 (I2b)
- new net: D61.1 (A1), J3.8 (Pin_8), U3.17 (I3b)
- new net: J4.2 (Pin_2), JP1.2 (B)
- new net: J4.4 (Pin_4), JP2.2 (B)
- new net: J4.6 (Pin_6), JP3.2 (B)
- new net: J4.8 (Pin_8), JP4.2 (B)
- no-connect marks 0 -> 6
Other:
- moved on the sheet: C1, C2, D1, D10, D11, D12, D13, D14, D15, D16, D17, D18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

Commit message: Finished routing. Added text.
Parts:
- added C12, C13: 10uF, Capacitor_SMD:C_0805_2012Metric, symbol Device:C_Small
- added H1, H2, H3, H4: MountingHole_Pad, MountingHole:MountingHole_3.2mm_M3_Pad_Via, symbol Mechanical:MountingHole_Pad
- C3, C4, C5, C6: value 47uF -> 330uF; footprint Capacitor_SMD:C_Elec_6.3x5.8 -> Capacitor_SMD:C_Elec_8x10.2
Connections:
- net GND: now also C12.2, C13.2, H1.1, H2.1, H3.1, H4.1
- net VCC: now also C12.1, C13.1
Changed lines of the file:
@@
 P 3250 2200
 F 0 "C4" H 3338 2246 50  0000 L CNN
-F 1 "47uF" H 3338 2155 50  0000 L CNN
-F 2 "Capacitor_SMD:C_Elec_6.3x5.8" H 3250 2200 50  0001 C CNN
+F 1 "330uF" H 3338 2155 50  0000 L CNN
+F 2 "Capacitor_SMD:C_Elec_8x10.2" H 3250 2200 50  0001 C CNN
 F 3 "~" H 3250 2200 50  0001 C CNN
 	1    3250 2200
@@
 P 2100 2450
 F 0 "C3" H 2188 2496 50  0000 L CNN
-F 1 "47uF" H 2188 2405 50  0000 L CNN
-F 2 "Capacitor_SMD:C_Elec_6.3x5.8" H 2100 2450 50  0001 C CNN
+F 1 "330uF" H 2188 2405 50  0000 L CNN
+F 2 "Capacitor_SMD:C_Elec_8x10.2" H 2100 2450 50  0001 C CNN
 F 3 "~" H 2100 2450 50  0001 C CNN
 	1    2100 2450
@@
 P 10800 2350
 F 0 "C5" H 10888 2396 50  0000 L CNN
-F 1 "47uF" H 10888 2305 50  0000 L CNN
-F 2 "Capacitor_SMD:C_Elec_6.3x5.8" H 10800 2350 50  0001 C CNN
+F 1 "330uF" H 10888 2305 50  0000 L CNN
+F 2 "Capacitor_SMD:C_Elec_8x10.2" H 10800 2350 50  0001 C CNN
 F 3 "~" H 10800 2350 50  0001 C CNN
 	1    10800 2350
@@
 P 11600 2100
 F 0 "C6" H 11688 2146 50  0000 L CNN
-F 1 "47uF" H 11688 2055 50  0000 L CNN
-F 2 "Capacitor_SMD:C_Elec_6.3x5.8" H 11600 2100 50  0001 C CNN
+F 1 "330uF" H 11688 2055 50  0000 L CNN
+F 2 "Capacitor_SMD:C_Elec_8x10.2" H 11600 2100 50  0001 C CNN
 F 3 "~" H 11600 2100 50  0001 C CNN
 	1    11600 2100
@@
 	-1   0    0    -1
 $EndComp
+$Comp
+L Device:C_Small C12
+U 1 1 5DB38982
+P 3800 3650
+F 0 "C12" H 3892 3696 50  0000 L CNN
+F 1 "10uF" H 3892 3605 50  0000 L CNN
+F 2 "Capacitor_SMD:C_0805_2012Metric" H 3800 3650 50  0001 C CNN
+F 3 "~" H 3800 3650 50  0001 C CNN
+	1    3800 3650
+	1    0    0    -1
+$EndComp
+Wire Wire Line
+	3800 3550 3800 3350
+Wire Wire Line
+	3800 3350 4150 3350
+Connection ~ 4150 3350
+$Comp
+L power:GND #PWR0103
+U 1 1 5DB96943
+P 3800 3800
+F 0 "#PWR0103" H 3800 3550 50  0001 C CNN
+F 1 "GND" H 3805 3627 50  0000 C CNN
+F 2 "" H 3800 3800 50  0001 C CNN
+F 3 "" H 3800 3800 50  0001 C CNN
+	1    3800 3800
+	1    0    0    -1
+$EndComp
+Wire Wire Line
+	3800 3800 3800 3750
+$Comp
+L Device:C_Small C13
+U 1 1 5DBF2E89
+P 10100 3650
+F 0 "C13" H 10192 3696 50  0000 L CNN
+F 1 "10uF" H 10192 3605 50  0000 L CNN
+F 2 "Capacitor_SMD:C_0805_2012Metric" H 10100 3650 50  0001 C CNN
+F 3 "~" H 10100 3650 50  0001 C CNN
+	1    10100 3650
+	1    0    0    -1
+$EndComp
+Wire Wire Line
+	10100 3550 10100 3350
+Wire Wire Line
+	10100 3350 10450 3350
+$Comp
+L power:GND #PWR0112
+U 1 1 5DBF2E91
+P 10100 3800
+F 0 "#PWR0112" H 10100 3550 50  0001 C CNN
+F 1 "GND" H 10105 3627 50  0000 C CNN
+F 2 "" H 10100 3800 50  0001 C CNN
+F 3 "" H 10100 3800 50  0001 C CNN
+	1    10100 3800
+	1    0    0    -1
+$EndComp
+Wire Wire Line
+	10100 3800 10100 3750
+$Comp
+L Mechanical:MountingHole_Pad H1
+U 1 1 5DFA8556
+P 900 10600
+F 0 "H1" H 950 10550 50  0000 L CNN
+F 1 "MountingHole_Pad" H 1000 10558 50  0001 L CNN
+F 2 "MountingHole:MountingHole_3.2mm_M3_Pad_Via" H 900 10600 50  0001 C CNN
+F 3 "~" H 900 10600 50  0001 C CNN
+	1    900  10600
+	1    0    0    -1
+$EndComp
+$Comp
+L power:GND #PWR0113
+U 1 1 5DFA8FC2
+P 900 10750
+F 0 "#PWR0113" H 900 10500 50  0001 C CNN
+F 1 "GND" H 905 10577 50  0000 C CNN
+F 2 "" H 900 10750 50  0001 C CNN
+F 3 "" H 900 10750 50  0001 C CNN
+	1    900  10750
+	1    0    0    -1
+$EndComp
+Wire Wire Line
+	900  10750 900  10700
+$Comp
+L Mechanical:MountingHole_Pad H2
+U 1 1 5E0084B0
+P 1150 10600
+F 0 "H2" H 1200 10550 50  0000 L CNN
+F 1 "MountingHole_Pad" H 1250 10558 50  0001 L CNN
+F 2 "MountingHole:MountingHole_3.2mm_M3_Pad_Via" H 1150 10600 50  0001 C CNN
+F 3 "~" H 1150 10600 50  0001 C CNN
+	1    1150 10600
+	1    0    0    -1
+$EndComp
+$Comp
+L power:GND #PWR0114
+U 1 1 5E0084B6
+P 1150 10750
+F 0 "#PWR0114" H 1150 10500 50  0001 C CNN
+F 1 "GND" H 1155 10577 50  0000 C CNN
+F 2 "" H 1150 10750 50  0001 C CNN
+F 3 "" H 1150 10750 50  0001 C CNN
+	1    1150 10750
+	1    0    0    -1
+$EndComp
+Wire Wire Line
+	1150 10750 1150 10700
+$Comp
+L Mechanical:MountingHole_Pad H3
+U 1 1 5E0657AB
+P 1400 10600
+F 0 "H3" H 1450 10550 50  0000 L CNN
+F 1 "MountingHole_Pad" H 1500 10558 50  0001 L CNN
+F 2 "MountingHole:MountingHole_3.2mm_M3_Pad_Via" H 1400 10600 50  0001 C CNN
+F 3 "~" H 1400 10600 50  0001 C CNN
+	1    1400 10600
+	1    0    0    -1
+$EndComp
+$Comp
+L power:GND #PWR0115
+U 1 1 5E0657B1
+P 1400 10750
+F 0 "#PWR0115" H 1400 10500 50  0001 C CNN
+F 1 "GND" H 1405 10577 50  0000 C CNN
+F 2 "" H 1400 10750 50  0001 C CNN
+F 3 "" H 1400 10750 50  0001 C CNN
+	1    1400 10750
+	1    0    0    -1
+$EndComp
+Wire Wire Line
+	1400 10750 1400 10700
+$Comp
+L Mechanical:MountingHole_Pad H4
+U 1 1 5E0C30FA
+P 1650 10600
+F 0 "H4" H 1700 10550 50  0000 L CNN
+F 1 "MountingHole_Pad" H 1750 10558 50  0001 L CNN
+F 2 "MountingHole:MountingHole_3.2mm_M3_Pad_Via" H 1650 10600 50  0001 C CNN
+F 3 "~" H 1650 10600 50  0001 C CNN
+	1    1650 10600
+	1    0    0    -1
+$EndComp
+$Comp
+L power:GND #PWR0116
+U 1 1 5E0C3100
+P 1650 10750
+F 0 "#PWR0116" H 1650 10500 50  0001 C CNN
+F 1 "GND" H 1655 10577 50  0000 C CNN
+F 2 "" H 1650 10750 50  0001 C CNN
+F 3 "" H 1650 10750 50  0001 C CNN
+	1    1650 10750
+	1    0    0    -1
+$EndComp
+Wire Wire Line
+	1650 10750 1650 10700
 $EndSCHEMATC
