File: Fancy-7-Segment-LED-Clock.kicad_pcb (KiCad board)
At the start: 2 copper layers, 115 x 180 mm, 64 parts, among them J1 Conn_02x04_Odd_Even, J3 Conn_02x04_Odd_Even, U1 TLC5952, U2 TLC5952

Commit message: ...
Parts:
- added J2: Conn_02x04_Odd_Even, ak:HARWIN_M20-7910842R, B.Cu at (171.6, 74.4)
- added J4: Conn_02x04_Odd_Even, ak:HARWIN_M20-7910842R, B.Cu at (42.5, 145.0)
- J1, J3: footprint ak:TE_5147722-3 -> ak:HARWIN_M20-8890845
- moved J1 25.8 mm to (155.5, 73.5), turned to 87 degrees
- moved J3 1.50 mm to (130.5, 145.0), turned to 87 degrees
Connections:
- U2 pad 30: (no net) -> Net-(J4-Pad2)

Commit message: ...
Parts:
- D1, D10, D11, D12, D13, D14, D15, D16, D17, D18, D19, D2, D20, D21, D22, D23, D24, D25, D26, D27, D28, D29, D3, D30, D31, D32, D33, D34, D35, D36, D37, D38, D39, D4, D40, D41, D42, D43, D44, D45, D46, D47, D48, D49, D5, D50, D51, D52, D53, D54, D55, D56, D6, D7, D8, D9: footprint ak:CREE_PLCC6_5.5x5.5 -> LED_SMD:LED_RGB_5050-6
- moved J2 126.4 mm to (45.2, 75.8)
- moved J1 22.1 mm to (133.5, 75.0)
- moved J4 10.9 mm to (41.2, 155.8)
- moved J3 10.1 mm to (129.2, 155.0)
- moved C1 3.00 mm to (83.0, 136.0)
- moved R2 3.00 mm to (79.0, 137.5)
- moved U2 3.00 mm to (83.5, 146.0)
- moved C2 2.00 mm to (86.5, 55.0)
- moved R1 2.00 mm to (82.0, 55.0)
- moved U1 2.00 mm to (86.5, 63.0)
- moved D1 0.50 mm to (93.0, 22.0), turned to 0 degrees
- moved D11 0.50 mm to (129.0, 39.5), turned to 90 degrees
- moved D12 0.50 mm to (129.5, 30.5), turned to 90 degrees
- moved D2 0.50 mm to (102.5, 22.0), turned to 0 degrees
- moved D3 0.50 mm to (112.0, 22.0), turned to 0 degrees
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Other:
- board size 115 x 180 mm -> 114 x 180 mm

Commit message: ...
Parts:
- added R10: R_Small, Resistors_SMD:R_0805, B.Cu at (75.0, 61.0)
- added R11: R_Small, Resistors_SMD:R_0805, B.Cu at (93.0, 147.5)
- added R12: R_Small, Resistors_SMD:R_0805, B.Cu at (93.0, 151.0)
- added R13: R_Small, Resistors_SMD:R_0805, B.Cu at (72.5, 151.5)
- added R14: R_Small, Resistors_SMD:R_0805, B.Cu at (72.5, 148.0)
- added R15: R_Small, Resistors_SMD:R_0805, B.Cu at (72.5, 144.5)
- added R16: R_Small, Resistors_SMD:R_0805, B.Cu at (72.5, 141.0)
- added R3: R_Small, Resistors_SMD:R_0805, B.Cu at (97.0, 59.5)
- added R4: R_Small, Resistors_SMD:R_0805, B.Cu at (97.0, 62.0)
- added R5: R_Small, Resistors_SMD:R_0805, B.Cu at (97.0, 64.5)
- added R6: R_Small, Resistors_SMD:R_0805, B.Cu at (97.0, 67.0)
- added R7: R_Small, Resistors_SMD:R_0805, B.Cu at (75.0, 68.5)
- added R8: R_Small, Resistors_SMD:R_0805, B.Cu at (75.0, 66.0)
- added R9: R_Small, Resistors_SMD:R_0805, B.Cu at (75.0, 63.5)
- moved D10 0.50 mm to (128.5, 49.5)
- moved D11 0.50 mm to (129.0, 40.0)
- moved D13 0.50 mm to (123.0, 152.0)
- moved D14 0.50 mm to (122.5, 161.5)
- moved D15 0.50 mm to (122.0, 171.0)
- moved D16 0.50 mm to (121.5, 180.5)
- moved D17 0.50 mm to (127.5, 68.5)
- moved D18 0.50 mm to (127.0, 78.0)
- moved D19 0.50 mm to (126.5, 87.5)
- moved D20 0.50 mm to (126.0, 97.0)
- moved D21 0.50 mm to (85.0, 189.0), turned to 0 degrees
- moved D22 0.50 mm to (94.5, 189.0), turned to 0 degrees
- moved D23 0.50 mm to (104.0, 189.0), turned to 0 degrees
- moved D24 0.50 mm to (113.5, 189.0), turned to 0 degrees
- moved D25 0.50 mm to (89.5, 105.5)
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Connections:
- U1 pad 11: Net-(D17-Pad3) -> Net-(R5-Pad2)
- U1 pad 14: Net-(D25-Pad3) -> Net-(R6-Pad2)
- U1 pad 17: Net-(D33-Pad3) -> Net-(R7-Pad2)
- U1 pad 20: Net-(D41-Pad3) -> Net-(R8-Pad2)
- U1 pad 23: Net-(D49-Pad3) -> Net-(R9-Pad2)
- U1 pad 26: Net-(D53-Pad3) -> Net-(R10-Pad2)
- U1 pad 5: Net-(D1-Pad3) -> Net-(R3-Pad2)
- U1 pad 8: Net-(D9-Pad3) -> Net-(R4-Pad2)
- U2 pad 11: Net-(D5-Pad3) -> Net-(R11-Pad2)
- U2 pad 16: Net-(D13-Pad1) -> Net-(R12-Pad2)
- U2 pad 17: Net-(D21-Pad3) -> Net-(R13-Pad2)
- U2 pad 20: Net-(D29-Pad3) -> Net-(R14-Pad2)
- U2 pad 23: Net-(D37-Pad3) -> Net-(R15-Pad2)
- U2 pad 26: Net-(D45-Pad3) -> Net-(R16-Pad2)
Routing:
- net (no net): track 0.00 -> 15.2 mm
- net Net-(D10-Pad3): track 0.00 -> 5.08 mm
- net Net-(D11-Pad4): track 0.00 -> 5.08 mm
- net Net-(D10-Pad4): track 0.00 -> 5.08 mm
- net Net-(D18-Pad6): track 0.00 -> 5.08 mm
- net Net-(D17-Pad6): track 0.00 -> 5.08 mm
- net Net-(D51-Pad4): track 0.00 -> 5.08 mm
- net Net-(D50-Pad4): track 0.00 -> 5.08 mm
- net Net-(D49-Pad4): track 0.00 -> 5.08 mm
- net Net-(D46-Pad4): track 0.00 -> 5.08 mm
- net Net-(D45-Pad4): track 0.00 -> 5.08 mm
- net Net-(D39-Pad6): track 0.00 -> 5.08 mm
- net Net-(D38-Pad6): track 0.00 -> 5.08 mm
- net Net-(D37-Pad6): track 0.00 -> 5.08 mm
- net Net-(D47-Pad4): track 0.00 -> 5.08 mm
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Other:
- net class Default: clearance 0.1 -> 0.15; trace_width 0.2 -> 0.15; via_dia 0.8 -> 0.6; via_drill 0.4 -> 0.3
- rule trace_clearance: 0.1 -> 0.15
- rule trace_min: 0.2 -> 0.15
- rule via_min_size: 0.4 -> 0.6

Commit message: ...
Parts:
- J3: footprint ak:HARWIN_M20-8890845 -> ak:HARWIN_M20-7910842R
- J4: footprint ak:HARWIN_M20-7910842R -> ak:HARWIN_M20-8890845
- moved J4 144.4 mm to (135.0, 46.0), turned to 87 degrees
- moved J3 136.0 mm to (46.8, 46.9), turned to 357 degrees
- moved J1 80.1 mm to (129.2, 155.0)
- moved J2 80.1 mm to (41.2, 155.8)
- moved C2 5.52 mm to (81.0, 54.5), turned to 90 degrees
- moved C1 5.22 mm to (78.0, 137.5), turned to 90 degrees
- moved R1 1.12 mm to (83.0, 54.5)
- moved R2 1.00 mm to (80.0, 137.5)
Connections:
- net Net-(J3-Pad4) renamed /SCLK
- net Net-(J3-Pad8) renamed /BLANK
- net Net-(U1-Pad30) renamed /SOUT_TO_SIN
- J3 pad 2: Net-(J3-Pad2) -> /LAT
- J3 pad 6: Net-(J3-Pad6) -> /SIN
- J4 pad 2: Net-(J4-Pad2) -> /LAT
- J4 pad 6: Net-(J3-Pad6) -> /SOUT
- U1 pad 2: Net-(J3-Pad2) -> /SIN
- U1 pad 4: Net-(J3-Pad6) -> /LAT
- U2 pad 30: Net-(J4-Pad2) -> /SOUT
- U2 pad 4: Net-(J3-Pad6) -> /LAT
Routing:
- net Vdrive: track 0.00 -> 556.1 mm
- net /BLANK: track 0.00 -> 279.8 mm, vias 0 -> 2
- net /SCLK: track 0.00 -> 266.0 mm, vias 0 -> 2
- net /LAT: track 0.00 -> 260.6 mm
- net /SOUT: track 0.00 -> 237.1 mm
- net /SOUT_TO_SIN: track 0.00 -> 89.8 mm, vias 0 -> 2
- net /SIN: track 0.00 -> 67.5 mm, vias 0 -> 2
- net Net-(D33-Pad1): track 0.00 -> 65.7 mm, vias 0 -> 1
- net Net-(D29-Pad1): track 0.00 -> 65.3 mm, vias 0 -> 1
- net Net-(D29-Pad2): track 0.00 -> 61.7 mm, vias 0 -> 1
- net Net-(D33-Pad2): track 0.00 -> 61.3 mm, vias 0 -> 1
- net Net-(D1-Pad1): track 0.00 -> 57.6 mm, vias 0 -> 1
- net Net-(D21-Pad2): track 0.00 -> 55.2 mm, vias 0 -> 1
- net Net-(D21-Pad1): track 0.00 -> 54.7 mm, vias 0 -> 1
- net Net-(D25-Pad3): track 0.00 -> 53.2 mm, vias 0 -> 1
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
Commit message: all change...
Parts:
- J1, J2: value Conn_02x04_Odd_Even -> Conn_02x04_Top_Bottom
- moved J1 26.5 mm to (127.8, 181.5)
- moved J2 26.5 mm to (39.8, 182.3)
- moved R7 8.31 mm to (83.0, 70.8), turned to 90 degrees
- moved R13 7.43 mm to (79.5, 154.0), turned to 90 degrees
- moved R14 7.21 mm to (76.5, 154.0), turned to 90 degrees
- moved R16 5.00 mm to (75.5, 145.0)
- moved R6 5.00 mm to (93.0, 70.0), turned to 90 degrees
- moved R15 4.61 mm to (75.5, 148.0)
- moved R8 4.03 mm to (78.5, 68.0)
- moved R9 3.81 mm to (78.5, 65.0)
- moved R10 3.64 mm to (78.5, 62.0)
- moved R4 2.50 mm to (95.0, 63.5)
- moved R5 2.50 mm to (95.0, 66.0)
- moved R3 2.24 mm to (95.0, 60.5)
- moved R11 2.06 mm to (91.0, 147.0)
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Connections:
- J1 pad 1: GND -> Vdrive
- J1 pad 4: Vdrive -> GND
- J1 pad 6: VCC -> GND
- J1 pad 7: GND -> VCC
- J2 pad 1: GND -> Vdrive
- J2 pad 4: Vdrive -> GND
- J2 pad 6: VCC -> GND
- J2 pad 7: GND -> VCC
Routing:
- net VCC: track 0.00 -> 286.6 mm, vias 0 -> 2
- net /BLANK: track 279.8 -> 207.8 mm, vias 2 -> 3
- net /SOUT: track 237.1 -> 169.9 mm, vias 0 -> 2
- net /LAT: track 260.6 -> 198.9 mm, vias 0 -> 3
- net /SCLK: track 266.0 -> 204.5 mm, vias 2 -> 3
- net Vdrive: track 556.1 -> 576.7 mm, vias 0 -> 2
- net Net-(D33-Pad1): track 65.7 -> 45.4 mm
- net Net-(D33-Pad2): track 61.3 -> 42.7 mm
- net Net-(D29-Pad1): track 65.3 -> 48.6 mm
- net Net-(D29-Pad3): track 49.4 -> 32.9 mm
- net Net-(D29-Pad2): track 61.7 -> 45.2 mm
- net Net-(D25-Pad3): track 53.2 -> 39.6 mm
- net Net-(D21-Pad1): track 54.7 -> 41.4 mm
- net Net-(D33-Pad3): track 46.1 -> 33.2 mm
- net Net-(D21-Pad2): track 55.2 -> 44.0 mm
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Other:
- board size 114 x 180 mm -> 114 x 183 mm
- net class Default: clearance 0.15 -> 0.2; trace_width 0.15 -> 0.2
- rule trace_clearance: 0.15 -> 0.2

Commit message: Routing...
Parts:
- moved R11 33.3 mm to (124.2, 144.5)
- moved R12 32.8 mm to (123.8, 151.5)
- moved R15 29.6 mm to (46.0, 149.8)
- moved R16 29.5 mm to (46.0, 146.5)
- moved R4 28.6 mm to (123.5, 60.8)
- moved R5 28.5 mm to (123.5, 64.5)
- moved R9 28.3 mm to (50.2, 63.0)
- moved R8 28.3 mm to (50.2, 67.8)
- moved R10 1.95 mm to (77.0, 60.8), turned to 270 degrees
- moved R3 0.25 mm to (95.0, 60.2)
Routing:
- net VCC: track 286.6 -> 345.2 mm, vias 2 -> 8
- net Net-(R11-Pad2): track 3.16 -> 37.4 mm
- net Net-(D5-Pad3): track 36.6 -> 3.64 mm
- net Net-(R12-Pad2): track 3.16 -> 35.9 mm
- net Net-(D37-Pad3): track 39.0 -> 8.02 mm
- net Net-(D13-Pad1): track 35.9 -> 5.14 mm
- net Net-(R15-Pad2): track 3.82 -> 34.0 mm
- net Net-(R16-Pad2): track 3.41 -> 33.5 mm
- net Net-(D9-Pad3): track 37.2 -> 7.81 mm
- net Net-(D49-Pad3): track 32.5 -> 3.17 mm
- net Net-(D17-Pad3): track 32.0 -> 2.92 mm
- net Net-(R4-Pad2): track 4.24 -> 33.2 mm
- net Net-(D41-Pad3): track 36.9 -> 8.52 mm
- net Net-(R9-Pad2): track 3.82 -> 32.1 mm
- net Net-(R8-Pad2): track 4.26 -> 32.4 mm
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- added copper zone on B.Cu, net GND
- added copper zone on B.Cu, net VCC
- added copper zone on B.Cu, net Vdrive
- added copper zone on F.Cu, net Vdrive

Commit message: Added line driver. Routing.
Parts:
- added C10: 100n, Capacitor_SMD:C_0805_2012Metric, B.Cu at (42.2, 161.2)
- added C11: 100n, Capacitor_SMD:C_0805_2012Metric, B.Cu at (43.8, 178.2)
- added C3: 47uF, Capacitor_SMD:C_Elec_6.3x5.8, B.Cu at (121.0, 162.0)
- added C4: 47uF, Capacitor_SMD:C_Elec_6.3x5.8, B.Cu at (121.0, 177.5)
- added C5: 47uF, Capacitor_SMD:C_Elec_6.3x5.8, B.Cu at (48.0, 165.2)
- added C6: 47uF, Capacitor_SMD:C_Elec_6.3x5.8, B.Cu at (48.0, 187.5)
- added C7: 100n, Capacitor_SMD:C_0805_2012Metric, B.Cu at (55.5, 26.5)
- added C8: 100n, Capacitor_SMD:C_0805_2012Metric, B.Cu at (117.5, 167.5)
- added C9: 100n, Capacitor_SMD:C_0805_2012Metric, B.Cu at (118.2, 183.5)
- added D57: D_TVS, Diode_SMD:D_SMA, B.Cu at (48.2, 159.5)
- added D58: 5V, Diode_SMD:D_SOD-323, B.Cu at (51.5, 43.5)
- added D59: 5V, Diode_SMD:D_SOD-323, B.Cu at (51.5, 39.0)
- added D60: 5V, Diode_SMD:D_SOD-323, B.Cu at (51.5, 34.5)
- added D61: 5V, Diode_SMD:D_SOD-323, B.Cu at (51.5, 30.0)
- added D62: D_TVS, Diode_SMD:D_SMA, B.Cu at (48.2, 181.8)
- added JP1: SolderJumper_2_Open, Jumper:SolderJumper-2_P1.3mm_Open_TrianglePad1.0x1.5mm, B.Cu at (94.0, 41.5)
- added JP2: SolderJumper_2_Open, Jumper:SolderJumper-2_P1.3mm_Open_TrianglePad1.0x1.5mm, B.Cu at (94.0, 38.5)
- added JP3: SolderJumper_2_Open, Jumper:SolderJumper-2_P1.3mm_Open_TrianglePad1.0x1.5mm, B.Cu at (94.0, 35.5)
- added JP4: SolderJumper_2_Open, Jumper:SolderJumper-2_P1.3mm_Open_TrianglePad1.0x1.5mm, B.Cu at (94.0, 32.8)
- added U3: 74LS244, Package_SO:SO-20_12.8x7.5mm_P1.27mm, B.Cu at (60.5, 36.0)
- C1, C2: value C_Small -> 100n
- J1: value Conn_02x04_Top_Bottom -> Power In
- J2: value Conn_02x04_Top_Bottom -> Power out
Connections:
- J3 pad 2: /LAT -> Net-(D58-Pad1)
- J3 pad 4: /SCLK -> Net-(D59-Pad1)
- J3 pad 6: /SIN -> Net-(D60-Pad1)
- J3 pad 8: /BLANK -> Net-(D61-Pad1)
- J4 pad 2: /LAT -> Net-(J4-Pad2)
- J4 pad 4: /SCLK -> Net-(J4-Pad4)
- J4 pad 6: /SOUT -> Net-(J4-Pad6)
- J4 pad 8: /BLANK -> Net-(J4-Pad8)
- U1 pad 33: Net-(U1-Pad33) -> GND
- U2 pad 33: Net-(U2-Pad33) -> GND
Routing:
- net VCC: track 345.2 -> 271.1 mm, vias 8 -> 6
- net Vdrive: track 569.5 -> 496.2 mm
- net /BLANK: track 208.9 -> 147.2 mm
- net /SCLK: track 209.3 -> 150.5 mm
- net /SOUT: track 170.6 -> 119.1 mm
- net /LAT: track 202.9 -> 152.1 mm
- net Net-(J4-Pad8): track 0.00 -> 43.1 mm
- net Net-(J4-Pad6): track 0.00 -> 41.7 mm
- net Net-(J4-Pad2): track 0.00 -> 40.9 mm
- net Net-(J4-Pad4): track 0.00 -> 40.6 mm
- net /SIN: track 74.7 -> 47.8 mm
- net Net-(D61-Pad1): track 0.00 -> 11.8 mm
- net Net-(D58-Pad1): track 0.00 -> 10.1 mm
- net Net-(D59-Pad1): track 0.00 -> 9.74 mm
- net Net-(D60-Pad1): track 0.00 -> 9.36 mm
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- added copper zone on F.Cu, net GND
Other:
- board size 114 x 183 mm -> 114.2 x 188 mm

Commit message: Routing. Via stitching
Parts:
- moved D62 8.16 mm to (41.0, 178.0), turned to 90 degrees
- moved C5 7.70 mm to (43.5, 159.0)
- moved D57 7.65 mm to (43.5, 165.5)
- moved C10 7.12 mm to (35.5, 159.0)
- moved J1 5.00 mm to (132.8, 181.5)
- moved J2 5.00 mm to (34.8, 182.3)
- moved J3 5.00 mm to (41.8, 46.9)
- moved J4 5.00 mm to (140.0, 46.0)
- moved D58 4.50 mm to (47.0, 43.5)
- moved D59 4.50 mm to (47.0, 39.0)
- moved D60 4.50 mm to (47.0, 34.5)
- moved D61 4.50 mm to (47.0, 30.0)
- moved C6 2.00 mm to (48.0, 185.5)
- moved C11 1.77 mm to (45.5, 178.5)
- moved C7 0.25 mm to (55.8, 26.5)
Routing:
- net Net-(J4-Pad6): track 41.7 -> 46.9 mm
- net Net-(D60-Pad1): track 9.36 -> 14.4 mm
- net Net-(D58-Pad1): track 10.1 -> 15.1 mm
- net Net-(D59-Pad1): track 9.74 -> 14.6 mm
- net Net-(J4-Pad2): track 40.9 -> 45.8 mm
- net Net-(J4-Pad4): track 40.6 -> 45.5 mm
- net Net-(J4-Pad8): track 43.1 -> 47.9 mm
- net Vdrive: track 496.2 -> 500.4 mm
- net Net-(D61-Pad1): track 11.8 -> 15.3 mm
- net GND: vias 0 -> 224
Other:
- board size 114.2 x 188 mm -> 125.2 x 213 mm
