File: Fancy-7-Segment-LED-Clock.kicad_pcb (KiCad board)
At the start: 2 copper layers, 125.2 x 213 mm, 100 parts, among them J1 Power In, J2 Power out, J3 Conn_02x04_Odd_Even, J4 Conn_02x04_Odd_Even, U1 TLC5952, U2 TLC5952, U3 74LS244

Commit message: Moved PCB and origin.
Parts:
- moved C1 41.7 mm to (111.0, 163.0)
- moved C10 41.7 mm to (68.5, 184.5)
- moved C11 41.7 mm to (78.5, 204.0)
- moved C2 41.7 mm to (114.0, 80.0)
- moved C3 41.7 mm to (154.0, 187.5)
- moved C4 41.7 mm to (154.0, 203.0)
- moved C5 41.7 mm to (76.5, 184.5)
- moved C6 41.7 mm to (81.0, 211.0)
- moved C7 41.7 mm to (88.8, 52.0)
- moved C8 41.7 mm to (150.5, 193.0)
- moved C9 41.7 mm to (151.2, 209.0)
- moved D1 41.7 mm to (126.0, 47.5)
- moved D10 41.7 mm to (161.5, 75.0)
- moved D11 41.7 mm to (162.0, 65.5)
- moved D12 41.7 mm to (162.5, 56.0)
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
Commit message: Square PCB
Parts:
- added C12: 10uF, Capacitor_SMD:C_0805_2012Metric, B.Cu at (112.0, 80.0)
- added C13: 10uF, Capacitor_SMD:C_0805_2012Metric, B.Cu at (109.0, 163.0)
- C3, C4, C5, C6: footprint Capacitor_SMD:C_Elec_6.3x5.8 -> Capacitor_SMD:C_Elec_8x10.2
- J3: value Conn_02x04_Odd_Even -> Signal in
- J4: value Conn_02x04_Odd_Even -> Signal out
- moved C9 10.8 mm to (160.5, 203.5), turned to 90 degrees
- moved C8 10.0 mm to (160.5, 193.1)
- moved C5 8.68 mm to (82.2, 191.0)
- moved J4 8.39 mm to (164.8, 70.0), turned to 90 degrees
- moved D60 7.83 mm to (73.0, 56.5)
- moved D61 7.43 mm to (73.0, 53.0)
- moved D58 7.35 mm to (73.0, 66.8)
- moved D59 7.11 mm to (73.0, 63.2)
- moved J3 6.21 mm to (69.0, 70.0), turned to 0 degrees
- moved C10 5.85 mm to (74.0, 186.5), turned to 90 degrees
- moved D57 3.20 mm to (74.0, 193.0), turned to 270 degrees
- moved J2 1.51 mm to (69.0, 207.0), turned to 0 degrees
- moved C6 1.00 mm to (82.0, 211.0)
- moved J1 1.00 mm to (164.8, 207.0), turned to 90 degrees
- moved C3 0.50 mm to (154.0, 187.0)
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Routing:
- net Vdrive: track 500.4 -> 519.1 mm
- net Net-(J4-Pad8): track 47.9 -> 39.2 mm
- net Net-(J4-Pad2): track 45.8 -> 37.2 mm
- net Net-(J4-Pad4): track 45.5 -> 37.7 mm
- net Net-(D61-Pad1): track 15.3 -> 23.0 mm
- net Net-(D60-Pad1): track 14.4 -> 21.8 mm
- net Net-(J4-Pad6): track 46.9 -> 39.7 mm
- net Net-(D59-Pad1): track 14.6 -> 20.8 mm
- net Net-(D58-Pad1): track 15.1 -> 20.1 mm
- net VCC: track 271.3 -> 272.9 mm
- net GND: vias 224 -> 227
Other:
- board size 125.2 x 213 mm -> 112 x 213 mm

Commit message: Finished routing. Added text.
Parts:
- added H1: MountingHole_Pad, MountingHole:MountingHole_3.2mm_M3_Pad_Via, F.Cu at (69.5, 31.5)
- added H2: MountingHole_Pad, MountingHole:MountingHole_3.2mm_M3_Pad_Via, F.Cu at (69.5, 230.5)
- added H3: MountingHole_Pad, MountingHole:MountingHole_3.2mm_M3_Pad_Via, F.Cu at (162.5, 230.5)
- added H4: MountingHole_Pad, MountingHole:MountingHole_3.2mm_M3_Pad_Via, F.Cu at (162.5, 31.5)
- C3, C4, C5, C6: value 47uF -> 330uF
- moved C10 5.00 mm to (79.0, 186.5)
- moved C11 5.00 mm to (83.5, 204.0)
- moved C5 5.00 mm to (87.2, 191.0)
- moved C6 5.00 mm to (87.0, 211.0)
- moved D57 5.00 mm to (79.0, 193.0)
- moved D62 5.00 mm to (79.0, 203.5)
- moved J2 5.00 mm to (74.0, 207.0)
- moved J3 5.00 mm to (74.0, 70.0)
- moved D58 4.00 mm to (77.0, 66.8)
- moved D59 4.00 mm to (77.0, 63.2)
- moved D60 4.00 mm to (77.0, 56.5)
- moved D61 4.00 mm to (77.0, 53.0)
- moved R11 1.25 mm to (156.0, 170.0)
- moved R12 0.75 mm to (156.0, 177.0)
Routing:
- net Vdrive: track 519.1 -> 496.5 mm
- net Net-(D59-Pad1): track 20.8 -> 15.8 mm
- net Net-(D61-Pad1): track 23.0 -> 18.0 mm
- net Net-(D60-Pad1): track 21.8 -> 16.8 mm
- net Net-(D58-Pad1): track 20.1 -> 15.1 mm
- net VCC: track 272.9 -> 268.8 mm
- net Net-(R11-Pad2): track 37.4 -> 36.1 mm
- net Net-(D13-Pad1): track 5.14 -> 6.14 mm
- net Net-(D5-Pad3): track 3.64 -> 4.61 mm
- net Net-(R12-Pad2): track 35.9 -> 35.1 mm
- net GND: vias 227 -> 204
Other:
- board size 112 x 213 mm -> 107 x 213 mm
- board text added: "BLANK"
- board text added: "CONTROL IN"
- board text added: "CONTROL OUT"
- board text added: "DC IN"
- board text added: "DC OUT"
- board text added: "LAT"
- board text added: "SCLK"
- board text added: "SIN"
- board text added: "SOUT"
- board text added: "VCC"
- board text added: "VLED"
