File: Digit_Colon/Digit_Colon.sch (KiCad schematic (older format))
At the start: 116 parts, among them J1 Power In, J2 Power out, J3 Signal in, J4 Signal out, U1 TLC5952, U2 TLC5952, U3 74LS244

Commit message: Minor changes. BOM
Parts:
- J1: value Power In -> DC IN
- J2: value Power out -> DC OUT
- R1, R10, R11, R12, R13, R14, R15, R16, R17, R18, R2, R3, R4, R5, R6, R7, R8, R9: value R_Small -> TBD
Connections:
- net VCC renamed +5VD
- net Vdrive renamed +15V
- no-connect marks 0 -> 4
Other:
- moved on the sheet: C1, C10, C11, C12, C13, C2, C3, C4, C5, C6, C7, C8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
