File: Digit_Colon/Digit_Colon.sch (KiCad schematic (older format))
At the start: 108 parts, among them J1 DC in, J2 DC out, J3 Signal in, J4 Signal out, U1 TLC5952, U2 TLC5952, U3 74LS244

Commit message: BOM update
Parts:
- J1: value DC in -> Conn_02x04_Odd_Even; Label (none) -> DC in
- J2: value DC out -> Conn_02x04_Odd_Even; Label (none) -> DC out
- J3: value Signal in -> Conn_02x04_Odd_Even; Label (none) -> Signal in
- J4: value Signal out -> Conn_02x04_Odd_Even; Label (none) -> Signal out
Changed lines of the file:
@@
 P 1200 8900
 F 0 "J1" H 1200 9100 50  0000 C CNN
-F 1 "DC in" H 1250 8600 50  0000 C CNN
+F 1 "Conn_02x04_Odd_Even" H 1250 8600 50  0001 C CNN
 F 2 "ak:HARWIN_M20-8890845" H 1200 8900 50  0001 C CNN
 F 3 "~" H 1200 8900 50  0001 C CNN
 F 4 "855-M20-8890845" H 1200 8900 50  0001 C CNN "Mouser"
+F 5 "DC in" H 1250 8600 50  0000 C CNN "Label"
 	1    1200 8900
 	1    0    0    -1
@@
 P 1150 3950
 F 0 "J3" H 1150 4150 50  0000 C CNN
-F 1 "Signal in" H 1250 3650 50  0000 C CNN
+F 1 "Conn_02x04_Odd_Even" H 1250 3650 50  0001 C CNN
 F 2 "ak:HARWIN_M20-7910842R" H 1150 3950 50  0001 C CNN
 F 3 "~" H 1150 3950 50  0001 C CNN
 F 4 "855-M20-7910842R" H 1150 3950 50  0001 C CNN "Mouser"
+F 5 "Signal in" H 1200 3650 50  0000 C CNN "Label"
 	1    1150 3950
 	1    0    0    -1
@@
 P 11600 8000
 F 0 "J4" H 11700 8200 50  0000 C CNN
-F 1 "Signal out" H 11600 7700 50  0000 C CNN
+F 1 "Conn_02x04_Odd_Even" H 11600 7700 50  0001 C CNN
 F 2 "ak:HARWIN_M20-8890845" H 11600 8000 50  0001 C CNN
 F 3 "~" H 11600 8000 50  0001 C CNN
 F 4 "855-M20-8890845" H 11600 8000 50  0001 C CNN "Mouser"
+F 5 "Signal out" H 11650 7700 50  0000 C CNN "Label"
 	1    11600 8000
 	-1   0    0    -1
@@
 P 15300 9050
 F 0 "J2" H 15350 9250 50  0000 C CNN
-F 1 "DC out" H 15350 8750 50  0000 C CNN
+F 1 "Conn_02x04_Odd_Even" H 15350 8750 50  0001 C CNN
 F 2 "ak:HARWIN_M20-7910842R" H 15300 9050 50  0001 C CNN
 F 3 "~" H 15300 9050 50  0001 C CNN
 F 4 "855-M20-7910842R" H 15300 9050 50  0001 C CNN "Mouser"
+F 5 "DC out" H 15350 8750 50  0000 C CNN "Label"
 	1    15300 9050
 	-1   0    0    -1

Commit message: Update
Parts:
- C1, C10, C11, C2, C7, C8, C9: Manufacturer (none) -> 08055C104KAT2A; Mouser 810-CGA3E2X7R1H104K -> (none); RS (none) -> 464-6688
- C12, C13: Manufacturer (none) -> C2012X7R1A106K125AC; RS (none) -> 788-3017
- C3, C4, C5, C6: Manufacturer (none) -> EEEFP1E331AP; RS (none) -> 568-525
- D57, D62: Manufacturer (none) -> SMAJ6.0CA-TR; RS (none) -> 795-8502
- D58, D59, D60, D61: RS (none) -> 187-1547
- R10, R11, R12, R13, R14, R15, R16, R17, R18, R3, R4, R5, R6, R7, R8, R9: Manufacturer (none) -> CRCW08050000Z0EA; RS (none) -> 679-0800
- U3: Manufacturer (none) -> SN74LS244DW; RS (none) -> 121-8344
Changed lines of the file:
@@
 EESchema Schematic File Version 4
-LIBS:Digit_Colon-cache
-EELAYER 29 0
+EELAYER 30 0
 EELAYER END
 $Descr A3 16535 11693
@@
 F 2 "Capacitor_SMD:C_0805_2012Metric" H 4350 2800 50  0001 C CNN
 F 3 "~" H 4350 2800 50  0001 C CNN
-F 4 "810-CGA3E2X7R1H104K " H 4350 2800 50  0001 C CNN "Mouser"
+F 4 "" H 4350 2800 50  0001 C CNN "Mouser"
+F 5 "08055C104KAT2A" H 4350 2800 50  0001 C CNN "Manufacturer"
+F 6 "464-6688" H 4350 2800 50  0001 C CNN "RS"
 	1    4350 2800
 	1    0    0    -1
@@
 F 2 "Capacitor_SMD:C_0805_2012Metric" H 10650 2800 50  0001 C CNN
 F 3 "~" H 10650 2800 50  0001 C CNN
-F 4 "810-CGA3E2X7R1H104K " H 10650 2800 50  0001 C CNN "Mouser"
+F 4 "" H 10650 2800 50  0001 C CNN "Mouser"
+F 5 "08055C104KAT2A" H 10650 2800 50  0001 C CNN "Manufacturer"
+F 6 "464-6688" H 10650 2800 50  0001 C CNN "RS"
 	1    10650 2800
 	1    0    0    -1
@@
 F 3 "~" H 7150 950 50  0001 C CNN
 F 4 "603-RT0805DRE071K58L" H 7150 950 50  0001 C CNN "Mouser"
+F 5 "CRCW08050000Z0EA" H 7150 950 50  0001 C CNN "Manufacturer"
+F 6 "679-0800" H 7150 950 50  0001 C CNN "RS"
 	1    7150 950
 	0    1    1    0
@@
 F 3 "~" H 7150 1800 50  0001 C CNN
 F 4 "603-RT0805DRE071K58L" H 7150 1800 50  0001 C CNN "Mouser"
+F 5 "CRCW08050000Z0EA" H 7150 1800 50  0001 C CNN "Manufacturer"
+F 6 "679-0800" H 7150 1800 50  0001 C CNN "RS"
 	1    7150 1800
 	0    1    1    0
@@
 F 3 "~" H 7150 2650 50  0001 C CNN
 F 4 "603-RT0805DRE071K58L" H 7150 2650 50  0001 C CNN "Mouser"
+F 5 "CRCW08050000Z0EA" H 7150 2650 50  0001 C CNN "Manufacturer"
+F 6 "679-0800" H 7150 2650 50  0001 C CNN "RS"
 	1    7150 2650
 	0    1    1    0
@@
 F 3 "~" H 7150 3500 50  0001 C CNN
 F 4 "603-RT0805DRE071K58L" H 7150 3500 50  0001 C CNN "Mouser"
+F 5 "CRCW08050000Z0EA" H 7150 3500 50  0001 C CNN "Manufacturer"
+F 6 "679-0800" H 7150 3500 50  0001 C CNN "RS"
 	1    7150 3500
 	0    1    1    0
@@
 F 3 "~" H 7150 4400 50  0001 C CNN
 F 4 "603-RT0805DRE071K58L" H 7150 4400 50  0001 C CNN "Mouser"
+F 5 "CRCW08050000Z0EA" H 7150 4400 50  0001 C CNN "Manufacturer"
+F 6 "679-0800" H 7150 4400 50  0001 C CNN "RS"
 	1    7150 4400
 	0    1    1    0
@@
 F 3 "~" H 7150 5250 50  0001 C CNN
 F 4 "603-RT0805DRE071K58L" H 7150 5250 50  0001 C CNN "Mouser"
+F 5 "CRCW08050000Z0EA" H 7150 5250 50  0001 C CNN "Manufacturer"
+F 6 "679-0800" H 7150 5250 50  0001 C CNN "RS"
 	1    7150 5250
 	0    1    1    0
@@
 F 3 "~" H 7150 6100 50  0001 C CNN
 F 4 "603-RT0805DRE071K58L" H 7150 6100 50  0001 C CNN "Mouser"
+F 5 "CRCW08050000Z0EA" H 7150 6100 50  0001 C CNN "Manufacturer"
+F 6 "679-0800" H 7150 6100 50  0001 C CNN "RS"
 	1    7150 6100
 	0    1    1    0
@@
 F 3 "~" H 7150 6950 50  0001 C CNN
 F 4 "603-RT0805DRE071K58L" H 7150 6950 50  0001 C CNN "Mouser"
+F 5 "CRCW08050000Z0EA" H 7150 6950 50  0001 C CNN "Manufacturer"
+F 6 "679-0800" H 7150 6950 50  0001 C CNN "RS"
 	1    7150 6950
 	0    1    1    0
@@
 F 3 "~" H 13600 3500 50  0001 C CNN
 F 4 "603-RT0805DRE071K58L" H 13600 3500 50  0001 C CNN "Mouser"
+F 5 "CRCW08050000Z0EA" H 13600 3500 50  0001 C CNN "Manufacturer"
+F 6 "679-0800" H 13600 3500 50  0001 C CNN "RS"
 	1    13600 3500
 	0    1    1    0
@@
 F 3 "~" H 13600 4400 50  0001 C CNN
 F 4 "603-RT0805DRE071K58L" H 13600 4400 50  0001 C CNN "Mouser"
+F 5 "CRCW08050000Z0EA" H 13600 4400 50  0001 C CNN "Manufacturer"
+F 6 "679-0800" H 13600 4400 50  0001 C CNN "RS"
 	1    13600 4400
 	0    1    1    0
@@
 F 3 "~" H 13600 5250 50  0001 C CNN
 F 4 "603-RT0805DRE071K58L" H 13600 5250 50  0001 C CNN "Mouser"
+F 5 "CRCW08050000Z0EA" H 13600 5250 50  0001 C CNN "Manufacturer"
+F 6 "679-0800" H 13600 5250 50  0001 C CNN "RS"
 	1    13600 5250
 	0    1    1    0
@@
 F 3 "~" H 13600 6100 50  0001 C CNN
 F 4 "603-RT0805DRE071K58L" H 13600 6100 50  0001 C CNN "Mouser"
+F 5 "CRCW08050000Z0EA" H 13600 6100 50  0001 C CNN "Manufacturer"
+F 6 "679-0800" H 13600 6100 50  0001 C CNN "RS"
 	1    13600 6100
 	0    1    1    0
@@
 F 3 "~" H 13600 6950 50  0001 C CNN
 F 4 "603-RT0805DRE071K58L" H 13600 6950 50  0001 C CNN "Mouser"
+F 5 "CRCW08050000Z0EA" H 13600 6950 50  0001 C CNN "Manufacturer"
+F 6 "679-0800" H 13600 6950 50  0001 C CNN "RS"
 	1    13600 6950
 	0    1    1    0
@@
 F 3 "~" H 13600 2650 50  0001 C CNN
 F 4 "603-RT0805DRE071K58L" H 13600 2650 50  0001 C CNN "Mouser"
+F 5 "CRCW08050000Z0EA" H 13600 2650 50  0001 C CNN "Manufacturer"
+F 6 "679-0800" H 13600 2650 50  0001 C CNN "RS"
 	1    13600 2650
 	0    1    1    0
@@
 F 3 "~" H 3400 9050 50  0001 C CNN
 F 4 "667-EEE-HA1E331UP " H 3400 9050 50  0001 C CNN "Mouser"
+F 5 "EEEFP1E331AP" H 3400 9050 50  0001 C CNN "Manufacturer"
+F 6 "568-525" H 3400 9050 50  0001 C CNN "RS"
 	1    3400 9050
 	1    0    0    -1
@@
 F 3 "~" H 2250 9300 50  0001 C CNN
 F 4 "667-EEE-HA1E331UP " H 2250 9300 50  0001 C CNN "Mouser"
+F 5 "EEEFP1E331AP" H 2250 9300 50  0001 C CNN "Manufacturer"
+F 6 "568-525" H 2250 9300 50  0001 C CNN "RS"
 	1    2250 9300
 	1    0    0    -1
@@
 F 2 "Capacitor_SMD:C_0805_2012Metric" H 3400 3100 50  0001 C CNN
 F 3 "~" H 3400 3100 50  0001 C CNN
-F 4 "810-CGA3E2X7R1H104K " H 3400 3100 50  0001 C CNN "Mouser"
+F 4 "" H 3400 3100 50  0001 C CNN "Mouser"
+F 5 "08055C104KAT2A" H 3400 3100 50  0001 C CNN "Manufacturer"
+F 6 "464-6688" H 3400 3100 50  0001 C CNN "RS"
 	1    3400 3100
 	0    -1   -1   0
@@
 F 3 "~" H 2050 4400 50  0001 C CNN
 F 4 "576-AQ05C-01FTG " H 2050 4400 50  0001 C CNN "Mouser"
+F 5 "187-1547" H 2050 4400 50  0001 C CNN "RS"
 	1    2050 4400
 	0    1    1    0
@@
 F 3 "~" H 2300 4400 50  0001 C CNN
 F 4 "576-AQ05C-01FTG " H 2300 4400 50  0001 C CNN "Mouser"
+F 5 "187-1547" H 2300 4400 50  0001 C CNN "RS"
 	1    2300 4400
 	0    1    1    0
@@
 F 3 "~" H 1800 9350 50  0001 C CNN
 F 4 "652-SMAJ6.0CA " H 1800 9350 50  0001 C CNN "Mouser"
+F 5 "SMAJ6.0CA-TR" H 1800 9350 50  0001 C CNN "Manufacturer"
+F 6 "795-8502" H 1800 9350 50  0001 C CNN "RS"
 	1    1800 9350
 	0    1    1    0
@@
 F 2 "Capacitor_SMD:C_0805_2012Metric" H 2600 9300 50  0001 C CNN
 F 3 "~" H 2600 9300 50  0001 C CNN
-F 4 "810-CGA3E2X7R1H104K " H 2600 9300 50  0001 C CNN "Mouser"
+F 4 "" H 2600 9300 50  0001 C CNN "Mouser"
+F 5 "08055C104KAT2A" H 2600 9300 50  0001 C CNN "Manufacturer"
+F 6 "464-6688" H 2600 9300 50  0001 C CNN "RS"
 	1    2600 9300
 	1    0    0    -1
@@
 F 2 "Capacitor_SMD:C_0805_2012Metric" H 3750 9050 50  0001 C CNN
 F 3 "~" H 3750 9050 50  0001 C CNN
-F 4 "810-CGA3E2X7R1H104K " H 3750 9050 50  0001 C CNN "Mouser"
+F 4 "" H 3750 9050 50  0001 C CNN "Mouser"
+F 5 "08055C104KAT2A" H 3750 9050 50  0001 C CNN "Manufacturer"
+F 6 "464-6688" H 3750 9050 50  0001 C CNN "RS"
 	1    3750 9050
 	1    0    0    -1
@@
 F 3 "~" H 3000 9050 50  0001 C CNN
 F 4 "652-SMAJ6.0CA " H 3000 9050 50  0001 C CNN "Mouser"
+F 5 "SMAJ6.0CA-TR" H 3000 9050 50  0001 C CNN "Manufacturer"
+F 6 "795-8502" H 3000 9050 50  0001 C CNN "RS"
 	1    3000 9050
 	0    1    1    0
@@
 F 3 "~" H 1800 4400 50  0001 C CNN
 F 4 "576-AQ05C-01FTG " H 1800 4400 50  0001 C CNN "Mouser"
+F 5 "187-1547" H 1800 4400 50  0001 C CNN "RS"
 	1    1800 4400
 	0    1    1    0
@@
 F 3 "~" H 1550 4400 50  0001 C CNN
 F 4 "576-AQ05C-01FTG " H 1550 4400 50  0001 C CNN "Mouser"
+F 5 "187-1547" H 1550 4400 50  0001 C CNN "RS"
 	1    1550 4400
 	0    1    1    0
@@
 F 2 "Capacitor_SMD:C_0805_2012Metric" H 13500 9150 50  0001 C CNN
 F 3 "~" H 13500 9150 50  0001 C CNN
-F 4 "810-CGA3E2X7R1H104K " H 13500 9150 50  0001 C CNN "Mouser"
+F 4 "" H 13500 9150 50  0001 C CNN "Mouser"
+F 5 "08055C104KAT2A" H 13500 9150 50  0001 C CNN "Manufacturer"
+F 6 "464-6688" H 13500 9150 50  0001 C CNN "RS"
 	1    13500 9150
 	-1   0    0    -1
@@
 F 2 "Capacitor_SMD:C_0805_2012Metric" H 14300 9400 50  0001 C CNN
 F 3 "~" H 14300 9400 50  0001 C CNN
-F 4 "810-CGA3E2X7R1H104K " H 14300 9400 50  0001 C CNN "Mouser"
+F 4 "" H 14300 9400 50  0001 C CNN "Mouser"
+F 5 "08055C104KAT2A" H 14300 9400 50  0001 C CNN "Manufacturer"
+F 6 "464-6688" H 14300 9400 50  0001 C CNN "RS"
 	1    14300 9400
 	-1   0    0    -1
@@
 F 3 "~" H 14700 9400 50  0001 C CNN
 F 4 "667-EEE-HA1E331UP " H 14700 9400 50  0001 C CNN "Mouser"
+F 5 "EEEFP1E331AP" H 14700 9400 50  0001 C CNN "Manufacturer"
+F 6 "568-525" H 14700 9400 50  0001 C CNN "RS"
 	1    14700 9400
 	-1   0    0    -1
@@
 F 3 "~" H 13900 9150 50  0001 C CNN
 F 4 "667-EEE-HA1E331UP " H 13900 9150 50  0001 C CNN "Mouser"
+F 5 "EEEFP1E331AP" H 13900 9150 50  0001 C CNN "Manufacturer"
+F 6 "568-525" H 13900 9150 50  0001 C CNN "RS"
 	1    13900 9150
 	-1   0    0    -1
@@
 F 3 "~" H 4000 2800 50  0001 C CNN
 F 4 "81-GRM21BR71A106KA3K" H 4000 2800 50  0001 C CNN "Mouser"
+F 5 "C2012X7R1A106K125AC" H 4000 2800 50  0001 C CNN "Manufacturer"
+F 6 "788-3017" H 4000 2800 50  0001 C CNN "RS"
 	1    4000 2800
 	1    0    0    -1
@@
 F 3 "~" H 10300 2800 50  0001 C CNN
 F 4 "81-GRM21BR71A106KA3K" H 10300 2800 50  0001 C CNN "Mouser"
+F 5 "C2012X7R1A106K125AC" H 10300 2800 50  0001 C CNN "Manufacturer"
+F 6 "788-3017" H 10300 2800 50  0001 C CNN "RS"
 	1    10300 2800
 	1    0    0    -1
@@
 F 3 "~" H 13600 1800 50  0001 C CNN
 F 4 "603-RT0805DRE071K58L" H 13600 1800 50  0001 C CNN "Mouser"
+F 5 "CRCW08050000Z0EA" H 13600 1800 50  0001 C CNN "Manufacturer"
+F 6 "679-0800" H 13600 1800 50  0001 C CNN "RS"
 	1    13600 1800
 	0    1    1    0
@@
 F 3 "~" H 13600 950 50  0001 C CNN
 F 4 "603-RT0805DRE071K58L" H 13600 950 50  0001 C CNN "Mouser"
+F 5 "CRCW08050000Z0EA" H 13600 950 50  0001 C CNN "Manufacturer"
+F 6 "679-0800" H 13600 950 50  0001 C CNN "RS"
 	1    13600 950
 	0    1    1    0
@@
 F 3 "http://www.ti.com/lit/gpn/sn74LS244" H 3200 3950 50  0001 C CNN
 F 4 "595-SN74LS244DWR" H 3200 3950 50  0001 C CNN "Mouser"
+F 5 "SN74LS244DW" H 3200 3950 50  0001 C CNN "Manufacturer"
+F 6 "121-8344" H 3200 3950 50  0001 C CNN "RS"
 	1    3200 3950
 	1    0    0    -1

Commit message: Minor changes
Parts:
- D57: RS 795-8502 -> 171-4263
- D62: value 6V TVS -> 16V TVS; Manufacturer SMAJ6.0CA-TR -> SMAJ16CA-E3/61; Mouser 652-SMAJ6.0CA -> (none); RS 795-8502 -> 814-1386
- R1, R2: value TBD -> 1k58; Mouser 71-CRCW08050000Z0EAC -> 603-RT0805DRE071K58L; RS (none) -> 123-1691
- R10, R11, R12, R13, R14, R15, R16, R17, R18, R3, R4, R5, R6, R7, R8, R9: Mouser 603-RT0805DRE071K58L -> (none)
Other:
- moved on the sheet: C1, C10, C11, C12, C4
