File: Digit_Colon/Digit_Colon.kicad_pcb (KiCad board)
At the start: 2 copper layers, 140.5 x 213 mm, 116 parts, among them J1 Power In, J2 Power out, J3 Signal in, J4 Signal out, U1 TLC5952, U2 TLC5952, U3 74LS244

Commit message: Ground vias digit+colon. Placement/routing controller
Parts:
- moved R6 1.75 mm to (126.0, 93.8)
Routing:
- net Net-(R6-Pad2): track 4.20 -> 3.16 mm
- net Net-(D25-Pad3): track 39.6 -> 40.7 mm
- net Vdrive: track 592.9 -> 593.7 mm
- net Net-(D25-Pad1): track 37.8 -> 37.2 mm
- net Net-(D25-Pad2): track 42.0 -> 41.4 mm
- net GND: vias 184 -> 282
- net (no net): vias 0 -> 1

Commit message: Minor changes. BOM
Parts:
- J1: value Power In -> DC IN
- J2: value Power out -> DC OUT
Connections:
- net VCC renamed +5VD
- net Vdrive renamed +15V
Routing:
- net GND: vias 282 -> 283
- net (no net): vias 1 -> 0

Commit message: Moved mounting holes. Moved stuff around on controller PCB.
Parts:
- moved H1 2.00 mm to (69.5, 33.5)
- moved H2 2.00 mm to (69.5, 228.5)
- moved H3 2.00 mm to (196.0, 228.5)
- moved H4 2.00 mm to (196.0, 33.5)
