File: Controller/Controller.sch (KiCad schematic (older format))
At the start: 94 parts, among them J1 CON_TLC, J2 CON_15V, J3 CON_ICSP, J4 DC out, J5 CON_5V, J6 CON_5V_AUX, J7 CON_USB_A, Q1 SI4435FDY, Q2 SI4435FDY, Q3 SQ2309ES, SW1 SW_Push, U1 FT232RL, U2 ATmega328P-AU, U3 DS3231M, U4 74AHC1G14, U5 MCP6001-OT, U6 MCP4012-xxxxCH, Y1 16MHz

Commit message: Replaced LDR with PD, changed USB connector.
Parts:
- removed R10: LDR07, OptoDevice:R_LDR_5.1x4.3mm_P3.4mm_Vertical, symbol Sensor_Optical:LDR07
- removed TP14, TP15: TestPoint_Alt, TestPoint:TestPoint_Loop_D2.60mm_Drill1.6mm_Beaded, symbol Connector:TestPoint_Alt
- removed U5: MCP6001-OT, Package_TO_SOT_SMD:SOT-23-5, symbol Amplifier_Operational:MCP6001-OT
- removed U6: MCP4012-xxxxCH, Package_TO_SOT_SMD:SOT-23-6, symbol Potentiometer_Digital:MCP4012-xxxxCH
- added JP1: 5V PASSTHRU, Connector_PinSocket_2.54mm:PinSocket_1x02_P2.54mm_Vertical, symbol Jumper:Jumper_2_Open
- added PD1: SFH 2440, OptoDevice:Osram_SMD-DIL2_4.5x4.0mm, symbol Sensor_Optical:SFH2440
- added R10, R18: ??, Resistor_SMD:R_0603_1608Metric, symbol Device:R_Small
- added U5: LMV301, Package_TO_SOT_SMD:SOT-353_SC-70-5, symbol ak:LMV301
- C23: value 10nF -> 1uF
- J7: footprint ak:UJ2-BV-1-TH -> Connector_USB:USB_B_TE_5787834_Vertical
- R15: value 47k -> ??
Connections:
- net labels added: PD_OUT
- net labels removed: LDR, POT_U~D~, ~POT_CS~
- wire segments 327 -> 329
Other:
- moved on the sheet: C21, C22, C23, C24, C25, R11, R12, R13, R15, SW1, TP16, U4

Commit message: shortened pcb by 1mm
Parts:
- J7: footprint Connector_USB:USB_B_TE_5787834_Vertical -> Connector_USB:USB_B_OST_USB-B1HSxx_Horizontal
- TP1, TP10, TP11, TP12, TP13, TP16, TP3, TP5, TP7, TP9: footprint TestPoint:TestPoint_Loop_D2.60mm_Drill1.6mm_Beaded -> TestPoint:TestPoint_Pad_D2.0mm
Changed lines of the file:
@@
 F 0 "J7" H 5900 5150 50  0000 C CNN
 F 1 "CON_USB_A" H 6300 4450 50  0000 C CNN
-F 2 "Connector_USB:USB_B_TE_5787834_Vertical" H 6200 4750 50  0001 C CNN
+F 2 "Connector_USB:USB_B_OST_USB-B1HSxx_Horizontal" H 6200 4750 50  0001 C CNN
 F 3 " ~" H 6200 4750 50  0001 C CNN
 	1    6050 4800
@@
 F 0 "TP16" V 10200 2600 50  0000 R CNN
 F 1 "TestPoint_Alt" H 10142 2367 50  0001 R CNN
-F 2 "TestPoint:TestPoint_Loop_D2.60mm_Drill1.6mm_Beaded" H 10400 2250 50  0001 C CNN
+F 2 "TestPoint:TestPoint_Pad_D2.0mm" H 10400 2250 50  0001 C CNN
 F 3 "~" H 10400 2250 50  0001 C CNN
 	1    10200 2250
@@
 F 0 "TP13" V 10200 2500 50  0000 R CNN
 F 1 "TestPoint_Alt" H 10142 2267 50  0001 R CNN
-F 2 "TestPoint:TestPoint_Loop_D2.60mm_Drill1.6mm_Beaded" H 10400 2150 50  0001 C CNN
+F 2 "TestPoint:TestPoint_Pad_D2.0mm" H 10400 2150 50  0001 C CNN
 F 3 "~" H 10400 2150 50  0001 C CNN
 	1    10200 2150
@@
 F 0 "TP12" V 10200 2400 50  0000 R CNN
 F 1 "TestPoint_Alt" H 10142 2167 50  0001 R CNN
-F 2 "TestPoint:TestPoint_Loop_D2.60mm_Drill1.6mm_Beaded" H 10400 2050 50  0001 C CNN
+F 2 "TestPoint:TestPoint_Pad_D2.0mm" H 10400 2050 50  0001 C CNN
 F 3 "~" H 10400 2050 50  0001 C CNN
 	1    10200 2050
@@
 F 0 "TP1" V 10200 1650 50  0000 R CNN
 F 1 "TestPoint_Alt" H 10142 1417 50  0001 R CNN
-F 2 "TestPoint:TestPoint_Loop_D2.60mm_Drill1.6mm_Beaded" H 10400 1300 50  0001 C CNN
+F 2 "TestPoint:TestPoint_Pad_D2.0mm" H 10400 1300 50  0001 C CNN
 F 3 "~" H 10400 1300 50  0001 C CNN
 	1    10200 1300
@@
 F 0 "TP3" V 10200 1750 50  0000 R CNN
 F 1 "TestPoint_Alt" H 10142 1517 50  0001 R CNN
-F 2 "TestPoint:TestPoint_Loop_D2.60mm_Drill1.6mm_Beaded" H 10400 1400 50  0001 C CNN
+F 2 "TestPoint:TestPoint_Pad_D2.0mm" H 10400 1400 50  0001 C CNN
 F 3 "~" H 10400 1400 50  0001 C CNN
 	1    10200 1400
@@
 F 0 "TP5" V 10200 1850 50  0000 R CNN
 F 1 "TestPoint_Alt" H 10142 1617 50  0001 R CNN
-F 2 "TestPoint:TestPoint_Loop_D2.60mm_Drill1.6mm_Beaded" H 10400 1500 50  0001 C CNN
+F 2 "TestPoint:TestPoint_Pad_D2.0mm" H 10400 1500 50  0001 C CNN
 F 3 "~" H 10400 1500 50  0001 C CNN
 	1    10200 1500
@@
 F 0 "TP7" V 10200 1950 50  0000 R CNN
 F 1 "TestPoint_Alt" H 10142 1717 50  0001 R CNN
-F 2 "TestPoint:TestPoint_Loop_D2.60mm_Drill1.6mm_Beaded" H 10400 1600 50  0001 C CNN
+F 2 "TestPoint:TestPoint_Pad_D2.0mm" H 10400 1600 50  0001 C CNN
 F 3 "~" H 10400 1600 50  0001 C CNN
 	1    10200 1600
@@
 F 0 "TP9" V 10200 2050 50  0000 R CNN
 F 1 "TestPoint_Alt" H 10142 1817 50  0001 R CNN
-F 2 "TestPoint:TestPoint_Loop_D2.60mm_Drill1.6mm_Beaded" H 10400 1700 50  0001 C CNN
+F 2 "TestPoint:TestPoint_Pad_D2.0mm" H 10400 1700 50  0001 C CNN
 F 3 "~" H 10400 1700 50  0001 C CNN
 	1    10200 1700
@@
 F 0 "TP10" V 10200 2150 50  0000 R CNN
 F 1 "TestPoint_Alt" H 10142 1917 50  0001 R CNN
-F 2 "TestPoint:TestPoint_Loop_D2.60mm_Drill1.6mm_Beaded" H 10400 1800 50  0001 C CNN
+F 2 "TestPoint:TestPoint_Pad_D2.0mm" H 10400 1800 50  0001 C CNN
 F 3 "~" H 10400 1800 50  0001 C CNN
 	1    10200 1800
@@
 F 0 "TP11" V 10200 2250 50  0000 R CNN
 F 1 "TestPoint_Alt" H 10142 2017 50  0001 R CNN
-F 2 "TestPoint:TestPoint_Loop_D2.60mm_Drill1.6mm_Beaded" H 10400 1900 50  0001 C CNN
+F 2 "TestPoint:TestPoint_Pad_D2.0mm" H 10400 1900 50  0001 C CNN
 F 3 "~" H 10400 1900 50  0001 C CNN
 	1    10200 1900

Commit message: BOM
Parts:
- C1, C11, C2, C9, U3: Mouser (none) -> 700-DS3231M+TRL
- C10, C12, C13, C15, C16, C18, C20, C27, C7, C8: Mouser (none) -> 576-1812L050PR
- C14, C17, C19, C6: Mouser (none) -> 710-885012206089
- C21, C22, C24: value 100n -> 100nF; Mouser (none) -> 576-1812L050PR
- C23: Mouser (none) -> 963-TMK107B7105MA-T
- C25: value 100n -> ??; Mouser (none) -> 576-1812L050PR
- C26: Mouser (none) -> 80-FC0H105ZFTBR44-SS
- C3: Mouser (none) -> 710-885012207092
- C4, C5: Mouser (none) -> 647-UUR1A101MCL1GS
- D1, D2: value BLUE -> LED blue; Mouser (none) -> 859-LTSTC193TBKT5A
- D3, D9: value SS1P3L -> MBR130; Mouser (none) -> 863-MBR130T1G
- D4: value ORANGE -> LED orange; Mouser (none) -> 859-LTST-C191KFKT
- D5: value GREEN -> LED green; Mouser (none) -> 859-LTST-C190KGKT
- D6: value RX ORANGE -> LED orange; Mouser (none) -> 859-LTST-C191KFKT
- D7: value TX GREEN -> LED green; Mouser (none) -> 859-LTST-C190KGKT
- D8: value RED -> LED red; Mouser (none) -> 859-LTST-C190KRKT
- F1: value 4A -> Fuse 4A; Mouser (none) -> 576-0154004.DRT
- F2: value 1A -> Fuse 1A; Mouser (none) -> 576-0154001.DR
- F3, F4: value 500mA -> Polyfuse 500mA; Mouser (none) -> 576-1812L050PR
- H1, H2: value MountingHole_Pad -> Mounting Hole
- J1: value CON_TLC -> DATA; Mouser (none) -> 855-M20-8890845
- J2: value CON_15V -> 15V
- J3: value CON_ICSP -> ICSP
- J4: value DC out -> DC OUT; Mouser (none) -> 855-M20-8890845
- J5: value CON_5V -> 5V
- J6: value CON_5V_AUX -> 5V AUX
- J7: value CON_USB_A -> USB
- L1, L2, L3: Mouser (none) -> 963-LBR2012T100K
- PD1: Mouser (none) -> 720-SFH2440
- Q1, Q2: Mouser (none) -> 78-SI4435FDY-T1-GE3
- Q3: Mouser (none) -> 781-SQ2309ES-T1_GE3
- SW1: value SW_Push -> RESET
- TP1: value TestPoint_Alt -> RTC_1PPS
- TP10: value TestPoint_Alt -> TLC_LAT
- TP11: value TestPoint_Alt -> TLC_BLANK
- TP12: value TestPoint_Alt -> +BATT
- TP13: value TestPoint_Alt -> VBUS
- TP16: value TestPoint_Alt -> +15V
- TP2, TP4: value TestPoint_Alt -> GND
- TP3: value TestPoint_Alt -> RTC_32K
- TP5: value TestPoint_Alt -> PD_OUT
- TP7: value TestPoint_Alt -> TLC_SDA
- TP9: value TestPoint_Alt -> TLC_SCL
- U1: Mouser (none) -> 895-FT232RL
- U2: Mouser (none) -> 556-ATMEGA328P-AU
- U4: Mouser (none) -> 595-SN74AHC1G14DBVR
- U5: Mouser (none) -> 926-LMV301MGX/NOPB
- Y1: Mouser (none) -> 81-CSTNE16M0V53Z000R
Connections:
- wire segments 329 -> 327
- no-connect marks 16 -> 18

Commit message: Replaced 15V connector. Created BOM and Gerbers
Parts:
- removed H1, H2: Mounting Hole, MountingHole:MountingHole_3.2mm_M3_Pad_Via, symbol Mechanical:MountingHole_Pad
- removed TP1: RTC_1PPS, TestPoint:TestPoint_Pad_D2.0mm, symbol Connector:TestPoint_Alt
- removed TP10: TLC_LAT, TestPoint:TestPoint_Pad_D2.0mm, symbol Connector:TestPoint_Alt
- removed TP11: TLC_BLANK, TestPoint:TestPoint_Pad_D2.0mm, symbol Connector:TestPoint_Alt
- removed TP12: +BATT, TestPoint:TestPoint_Pad_D2.0mm, symbol Connector:TestPoint_Alt
- removed TP13: VBUS, TestPoint:TestPoint_Pad_D2.0mm, symbol Connector:TestPoint_Alt
- removed TP16: +15V, TestPoint:TestPoint_Pad_D2.0mm, symbol Connector:TestPoint_Alt
- removed TP2, TP4: GND, TestPoint:TestPoint_Loop_D2.60mm_Drill1.6mm_Beaded, symbol Connector:TestPoint_Alt
- removed TP3: RTC_32K, TestPoint:TestPoint_Pad_D2.0mm, symbol Connector:TestPoint_Alt
- removed TP5: PD_OUT, TestPoint:TestPoint_Pad_D2.0mm, symbol Connector:TestPoint_Alt
- removed TP7: TLC_SDA, TestPoint:TestPoint_Pad_D2.0mm, symbol Connector:TestPoint_Alt
- removed TP9: TLC_SCL, TestPoint:TestPoint_Pad_D2.0mm, symbol Connector:TestPoint_Alt
- C1, C2: Mouser 700-DS3231M+TRL -> 661-EMVE250ADA331MJA
- C11, C9: Mouser 700-DS3231M+TRL -> 667-EEE-FK1K4R7P
- J2: footprint Connector_JST:JST_XH_B2B-XH-A_1x02_P2.50mm_Vertical -> Connectors_JST:JST_XH_B03B-XH-A_03x2.50mm_Straight; symbol Connector_Generic:Conn_01x02 -> Connector_Generic:Conn_01x03; Digikey (none) -> 455-2248-ND
- J3: Digikey (none) -> 732-5394-ND
- J5, J6: Digikey (none) -> 455-2247-ND
- J7: Mouser (none) -> 649-61729-0011BLF
- JP1: Digikey (none) -> S1012EC-02-ND
- R1, R13, R2, R3, R4, R5, R6, R7: Mouser (none) -> 660-RN73H1JT1001F100
- R11, R12: Mouser (none) -> 660-RN73H1JTD1002F50
- R14: Mouser (none) -> 660-RN73H1JT1000F100
- R16, R17, R8, R9: Mouser (none) -> 660-RN73H1JT4701F100
- U5: symbol ak:LMV301 -> Controller-rescue:LMV301-ak
- renumbered D9 to D1, D3 to D2, D1 to LD1, D2 to LD2, D4 to LD3, D5 to LD4, D6 to LD5, D7 to LD6, D8 to LD7
Connections:
- net labels added: Mounting Hole
- wire segments 327 -> 328

Commit message: BOM update
Parts:
- C25: Mouser 576-1812L050PR -> (none)
- J1: value DATA -> Conn_02x04_Top_Bottom; Label (none) -> Data
- J3: value ICSP -> Conn_02x03_Top_Bottom; Label (none) -> ICSP
- J4: value DC OUT -> Conn_02x04_Top_Bottom; Label (none) -> DC out
- J6: value 5V AUX -> Conn_01x02; Label (none) -> 5V aux
- J7: value USB -> USB_A
- JP1: value 5V PASSTHRU -> Jumper; Label (none) -> 5V passthrough
- LD3, LD5: value LED orange -> LED; Label (none) -> Orange
- LD4, LD6: value LED green -> LED; Label (none) -> Green
- LD7: value LED red -> LED; Label (none) -> Red
Changed lines of the file:
@@
 P 5700 1450
 F 0 "J1" H 5800 1650 50  0000 C CNN
-F 1 "DATA" H 5750 1150 50  0000 C CNN
+F 1 "Conn_02x04_Top_Bottom" H 5750 1150 50  0001 C CNN
 F 2 "ak:HARWIN_M20-8890845" H 5700 1450 50  0001 C CNN
 F 3 "~" H 5700 1450 50  0001 C CNN
 F 4 "855-M20-8890845 " H 5700 1450 50  0001 C CNN "Mouser"
+F 5 "Data" H 5750 1150 50  0000 C CNN "Label"
 	1    5700 1450
 	-1   0    0    -1
@@
 P 9800 5000
 F 0 "LD5" H 9950 5050 50  0000 C CNN
-F 1 "LED orange" H 9750 4850 50  0000 C CNN
+F 1 "LED" H 9750 4850 50  0001 C CNN
 F 2 "LED_SMD:LED_0603_1608Metric" H 9800 5000 50  0001 C CNN
 F 3 "~" H 9800 5000 50  0001 C CNN
 F 4 "859-LTST-C191KFKT" H 9800 5000 50  0001 C CNN "Mouser"
+F 5 "Orange" H 9850 4900 50  0000 C CNN "Label"
 	1    9800 5000
 	0    -1   -1   0
@@
 P 10200 5000
 F 0 "LD6" H 10350 5050 50  0000 C CNN
-F 1 "LED green" H 10150 4850 50  0000 C CNN
+F 1 "LED" H 10150 4850 50  0001 C CNN
 F 2 "LED_SMD:LED_0603_1608Metric" H 10200 5000 50  0001 C CNN
 F 3 "~" H 10200 5000 50  0001 C CNN
 F 4 "859-LTST-C190KGKT" H 10200 5000 50  0001 C CNN "Mouser"
+F 5 "Green" H 10250 4900 50  0000 C CNN "Label"
 	1    10200 5000
 	0    -1   -1   0
@@
 P 7700 1650
 F 0 "J3" H 7700 1850 50  0000 C CNN
-F 1 "ICSP" H 7750 1450 50  0000 C CNN
+F 1 "Conn_02x03_Top_Bottom" H 7750 1450 50  0001 C CNN
 F 2 "Connector_IDC:IDC-Header_2x03_P2.54mm_Vertical" H 7700 1650 50  0001 C CNN
 F 3 "~" H 7700 1650 50  0001 C CNN
 F 4 "732-5394-ND" H 7700 1650 50  0001 C CNN "Digikey"
+F 5 "ICSP" H 7750 1450 50  0000 C CNN "Label"
 	1    7700 1650
 	1    0    0    -1
@@
 P 14100 6150
 F 0 "LD7" H 14250 6200 50  0000 C CNN
-F 1 "LED red" H 14050 6000 50  0000 C CNN
+F 1 "LED" H 14050 6000 50  0001 C CNN
 F 2 "LED_SMD:LED_0603_1608Metric" H 14100 6150 50  0001 C CNN
 F 3 "~" H 14100 6150 50  0001 C CNN
 F 4 "859-LTST-C190KRKT" H 14100 6150 50  0001 C CNN "Mouser"
+F 5 "Red" H 14100 6050 50  0000 C CNN "Label"
 	1    14100 6150
 	0    -1   -1   0
@@
 P 6050 4800
 F 0 "J7" H 5900 5150 50  0000 C CNN
-F 1 "USB" H 6300 4450 50  0000 C CNN
+F 1 "USB_A" H 6300 4450 50  0000 C CNN
 F 2 "Connector_USB:USB_B_OST_USB-B1HSxx_Horizontal" H 6200 4750 50  0001 C CNN
 F 3 " ~" H 6200 4750 50  0001 C CNN
@@
 P 4250 4600
 F 0 "LD4" H 4400 4650 50  0000 C CNN
-F 1 "LED green" H 4200 4450 50  0000 C CNN
+F 1 "LED" H 4200 4450 50  0001 C CNN
 F 2 "LED_SMD:LED_0603_1608Metric" H 4250 4600 50  0001 C CNN
 F 3 "~" H 4250 4600 50  0001 C CNN
 F 4 "859-LTST-C190KGKT" H 4250 4600 50  0001 C CNN "Mouser"
+F 5 "Green" H 4350 4500 50  0000 C CNN "Label"
 	1    4250 4600
 	0    -1   -1   0
@@
 P 3300 4600
 F 0 "LD3" H 3450 4650 50  0000 C CNN
-F 1 "LED orange" H 3250 4450 50  0000 C CNN
+F 1 "LED" H 3250 4450 50  0001 C CNN
 F 2 "LED_SMD:LED_0603_1608Metric" H 3300 4600 50  0001 C CNN
 F 3 "~" H 3300 4600 50  0001 C CNN
 F 4 "859-LTST-C191KFKT" H 3300 4600 50  0001 C CNN "Mouser"
+F 5 "Orange" H 3400 4500 50  0000 C CNN "Label"
 	1    3300 4600
 	0    -1   -1   0
@@
 P 3900 1750
 F 0 "J4" H 3950 1950 50  0000 C CNN
-F 1 "DC OUT" H 3950 1450 50  0000 C CNN
+F 1 "Conn_02x04_Top_Bottom" H 3950 1450 50  0001 C CNN
 F 2 "ak:HARWIN_M20-8890845" H 3900 1750 50  0001 C CNN
 F 3 "~" H 3900 1750 50  0001 C CNN
 F 4 "855-M20-8890845 " H 3900 1750 50  0001 C CNN "Mouser"
+F 5 "DC out" H 3950 1450 50  0000 C CNN "Label"
 	1    3900 1750
 	1    0    0    -1
@@
 P 1150 4050
 F 0 "J6" H 1150 4250 50  0000 C CNN
-F 1 "5V AUX" H 1050 4150 50  0000 C CNN
+F 1 "Conn_01x02" H 1050 4150 50  0001 C CNN
 F 2 "Connector_JST:JST_XH_B2B-XH-A_1x02_P2.50mm_Vertical" H 1150 4050 50  0001 C CNN
 F 3 "~" H 1150 4050 50  0001 C CNN
 F 4 "455-2247-ND" H 1150 4050 50  0001 C CNN "Digikey"
+F 5 "5V aux" H 1150 3850 50  0000 C CNN "Label"
 	1    1150 4050
 	-1   0    0    -1
@@
 F 2 "Capacitor_SMD:C_0603_1608Metric" H 2850 7700 50  0001 C CNN
 F 3 "~" H 2850 7700 50  0001 C CNN
-F 4 "576-1812L050PR" H 2850 7700 50  0001 C CNN "Mouser"
 	1    2850 7700
 	0    1    -1   0
@@
 P 3900 2850
 F 0 "JP1" H 3900 3000 50  0000 C CNN
-F 1 "5V PASSTHRU" H 3900 2750 50  0000 C CNN
+F 1 "Jumper" H 3900 2750 50  0001 C CNN
 F 2 "Connector_PinSocket_2.54mm:PinSocket_1x02_P2.54mm_Vertical" H 3900 2850 50  0001 C CNN
 F 3 "~" H 3900 2850 50  0001 C CNN
 F 4 "S1012EC-02-ND" H 3900 2850 50  0001 C CNN "Digikey"
+F 5 "5V passthrough" H 3900 2750 50  0000 C CNN "Label"
 	1    3900 2850
 	1    0    0    -1
