File: Power_Supply/Power supply.sch (KiCad schematic (older format))
At the start: 29 parts

Commit message: Power supply
Parts:
- removed C? (x3): 10uF, symbol Device:CP_Small
- removed D?: Q_SCR_KAG, symbol Device:Q_SCR_KAG
- removed D?: D, symbol Device:D
- removed TR?: TRANSF6, symbol Transformer:TRANSF6
- added C6, C8, C9: 10uF, Capacitor_THT:CP_Radial_D5.0mm_P2.00mm, symbol Device:CP_Small
- added D1, D6: 1N5819, Diode_THT:D_DO-41_SOD81_P10.16mm_Horizontal, symbol Diode:1N5819
- added D5, D8: 1N4148, Diode_THT:D_DO-35_SOD27_P7.62mm_Horizontal, symbol Diode:1N4148
- added J1, J2, J3, J4, J5, J6, J7, J8, J9: Conn_01x01, Connector_Pin:Pin_D1.0mm_L10.0mm, symbol Connector_Generic:Conn_01x01
- added J10: Conn_01x04, Connector_PinHeader_2.54mm:PinHeader_1x04_P2.54mm_Vertical, symbol Connector_Generic:Conn_01x04
- C1: renamed from C?; footprint (none) -> Capacitor_THT:CP_Radial_D25.0mm_P10.00mm_SnapIn; Manufacturer LGU1V472MELA -> LGU1V472MELA; RS 846-6931 -> 846-6931
- C10, C7: renamed from C?; footprint (none) -> Capacitor_THT:C_Disc_D5.0mm_W2.5mm_P2.50mm
- C2, C3, C4: renamed from C?; footprint (none) -> Capacitor_THT:CP_Radial_D25.0mm_P10.00mm_SnapIn
- C5: renamed from C?; footprint (none) -> Capacitor_THT:CP_Radial_D5.0mm_P2.00mm; Manufacturer (none) -> UPW1V100MDD; RS (none) -> 715-2713
- D2: renamed from D?; footprint (none) -> Diode_THT:Diode_Bridge_Vishay_GBU
- D3: renamed from D?; value 13V -> 12V; footprint (none) -> Diode_THT:D_DO-35_SOD27_P7.62mm_Horizontal
- D4: renamed from D?; footprint (none) -> Package_TO_SOT_THT:TO-220F-3_Horizontal_TabDown
- D7: renamed from D?; value 6V -> 5V; footprint (none) -> Diode_THT:D_DO-35_SOD27_P7.62mm_Horizontal
- F1: renamed from F?; footprint (none) -> Fuse:Fuseholder_Cylinder-5x20mm_Schurter_0031_8201_Horizontal_Open
- R1, R2, R3, R4, R5, R6, R7, R8: renamed from R?; footprint (none) -> Resistor_THT:R_Axial_DIN0207_L6.3mm_D2.5mm_P10.16mm_Horizontal
- RV1: renamed from RV?; value Varistor -> S20K275; footprint (none) -> Varistor:RV_Disc_D21.5mm_W5.4mm_P10mm; Manufacturer (none) -> B72220S0271K101; RS (none) -> 204-2208
- U1, U2: renamed from U?; footprint (none) -> Package_TO_SOT_THT:TO-220-3_Vertical
Connections:
- net labels added: +12V, +5V, Earth_Protective
- wire segments 112 -> 131
Other:
- note added: "Trafo RS 671-8987\nCase Hammond 1598 Series"
- note removed: "Trafo RS 671-8987"
- moved on the sheet: C10, D4, D7, R5, R6, R7, R8, U2
