File: Power_Supply/Power supply.sch (KiCad schematic (older format))
At the start: 40 parts, among them J1 Conn_01x01, J10 Conn_01x04, J2 Conn_01x01, J3 Conn_01x01, J4 Conn_01x01, J5 Conn_01x01, J6 Conn_01x01, J7 Conn_01x01, J8 Conn_01x01, J9 Conn_01x01, U1 LM1084-ADJ, U2 LM1084-ADJ

Commit message: Power supply
Parts:
- C2, C3, C4: Manufacturer LGU1V472MELA -> LGU1V472MELA; RS 846-6931 -> 846-6931
- D1, D6: Manufacturer (none) -> 1N5819; RS (none) -> 486-4460
- D2: Manufacturer GBU1006 -> GBU1006; RS 923-5457 -> 923-5457
- D4: RS 177-5215 -> 862-4950
Changed lines of the file:
@@
 F 2 "Diode_THT:Diode_Bridge_Vishay_GBU" H 3000 2150 50  0001 C CNN
 F 3 "~" H 3000 2150 50  0001 C CNN
-F 4 " GBU1006 " H 3000 2150 50  0001 C CNN "Manufacturer"
-F 5 " 923-5457" H 3000 2150 50  0001 C CNN "RS"
+F 4 "GBU1006 " H 3000 2150 50  0001 C CNN "Manufacturer"
+F 5 "923-5457" H 3000 2150 50  0001 C CNN "RS"
 	1    3000 2150
 	1    0    0    -1
@@
 F 2 "Capacitor_THT:CP_Radial_D25.0mm_P10.00mm_SnapIn" H 4538 2350 50  0001 C CNN
 F 3 "~" H 4500 2500 50  0001 C CNN
-F 4 " LGU1V472MELA " H 4500 2500 50  0001 C CNN "Manufacturer"
-F 5 " 846-6931" H 4500 2500 50  0001 C CNN "RS"
+F 4 "LGU1V472MELA " H 4500 2500 50  0001 C CNN "Manufacturer"
+F 5 "846-6931" H 4500 2500 50  0001 C CNN "RS"
 	1    4500 2500
 	1    0    0    -1
@@
 F 2 "Capacitor_THT:CP_Radial_D25.0mm_P10.00mm_SnapIn" H 5038 2350 50  0001 C CNN
 F 3 "~" H 5000 2500 50  0001 C CNN
-F 4 " LGU1V472MELA " H 5000 2500 50  0001 C CNN "Manufacturer"
-F 5 " 846-6931" H 5000 2500 50  0001 C CNN "RS"
+F 4 "LGU1V472MELA " H 5000 2500 50  0001 C CNN "Manufacturer"
+F 5 "846-6931" H 5000 2500 50  0001 C CNN "RS"
 	1    5000 2500
 	1    0    0    -1
@@
 F 2 "Capacitor_THT:CP_Radial_D25.0mm_P10.00mm_SnapIn" H 5538 2350 50  0001 C CNN
 F 3 "~" H 5500 2500 50  0001 C CNN
-F 4 " LGU1V472MELA " H 5500 2500 50  0001 C CNN "Manufacturer"
-F 5 " 846-6931" H 5500 2500 50  0001 C CNN "RS"
+F 4 "LGU1V472MELA " H 5500 2500 50  0001 C CNN "Manufacturer"
+F 5 "846-6931" H 5500 2500 50  0001 C CNN "RS"
 	1    5500 2500
 	1    0    0    -1
@@
 F 3 "~" V 9800 2450 50  0001 C CNN
 F 4 "MCR72-6G" H 9800 2450 50  0001 C CNN "Manufacturer"
-F 5 "177-5215" H 9800 2450 50  0001 C CNN "RS"
+F 5 "862-4950" H 9800 2450 50  0001 C CNN "RS"
 	1    9800 2450
 	1    0    0    -1
@@
 F 2 "Diode_THT:D_DO-41_SOD81_P10.16mm_Horizontal" H 6850 1575 50  0001 C CNN
 F 3 "http://www.vishay.com/docs/88525/1n5817.pdf" H 6850 1750 50  0001 C CNN
+F 4 "1N5819 " H 6850 1750 50  0001 C CNN "Manufacturer"
+F 5 "486-4460" H 6850 1750 50  0001 C CNN "RS"
 	1    6850 1750
 	1    0    0    -1
@@
 F 2 "Diode_THT:D_DO-41_SOD81_P10.16mm_Horizontal" H 6850 3375 50  0001 C CNN
 F 3 "http://www.vishay.com/docs/88525/1n5817.pdf" H 6850 3550 50  0001 C CNN
+F 4 "1N5819 " H 6850 3550 50  0001 C CNN "Manufacturer"
+F 5 "486-4460" H 6850 3550 50  0001 C CNN "RS"
 	1    6850 3550
 	1    0    0    -1

Commit message: psu
Parts:
- removed F1: Fuse, Fuse:Fuseholder_Cylinder-5x20mm_Schurter_0031_8201_Horizontal_Open, symbol Device:Fuse
- removed J2, J3, J6, J7, J9: Conn_01x01, Connector_Pin:Pin_D1.0mm_L10.0mm, symbol Connector_Generic:Conn_01x01
- removed R1, R3: ?, Resistor_THT:R_Axial_DIN0207_L6.3mm_D2.5mm_P10.16mm_Horizontal, symbol Device:R_Small
- removed RV1: S20K275, Varistor:RV_Disc_D21.5mm_W5.4mm_P10mm, symbol Device:Varistor
- added C11: 10uF, Capacitor_THT:CP_Radial_D5.0mm_P2.00mm, symbol Device:CP_Small
- added C12, C13: 100nF, Capacitor_THT:C_Disc_D5.0mm_W2.5mm_P2.50mm, symbol Device:C_Small
- added D8: 1N4148, Diode_THT:D_DO-35_SOD27_P7.62mm_Horizontal, symbol Diode:1N4148
- added K1: RY611012, ak:RY611012, symbol ak:RY611012
- added Q1: BC548, Package_TO_SOT_THT:TO-92_Inline, symbol Transistor_BJT:BC337
- added R4: 100k, Resistor_THT:R_Axial_DIN0207_L6.3mm_D2.5mm_P10.16mm_Horizontal, symbol Device:R_Small
- added TH1: 5R, Varistor:RV_Disc_D21.5mm_W6.1mm_P7.5mm, symbol Device:Thermistor_NTC
- added U3: NE555P, Package_DIP:DIP-8_W7.62mm, symbol Timer:NE555P
- R5: value ? -> 100k
- R7: value ? -> 10k
- U1: value LM1084-ADJ -> LM1084-12
- U2: value LM1084-ADJ -> LM1084-5
- renumbered D8 to D9, J4 to J2, J5 to J3, J8 to J4, J10 to J5, R2 to R1, R4 to R2, R6 to R3, R8 to R6
Connections:
- net labels added: VDC
- net labels removed: Earth_Protective
- wire segments 131 -> 149
Other:
- note removed: "Trafo RS 671-8987\nCase Hammond 1598 Series"
- moved on the sheet: C1, C10, C2, C3, C4, C5, C6, C7, C8, C9, D1, D2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

Commit message: PSU
Parts:
- added F1: 3A, Fuse:Fuseholder_Cylinder-5x20mm_Schurter_0031_8201_Horizontal_Open, symbol Device:Fuse
- added HS1: Heatsink, ak:HS-160x50, symbol Mechanical:Heatsink
- U3: symbol Timer:NE555P -> Power-supply-rescue:NE555P-Timer
Connections:
- wire segments 149 -> 150
Changed lines of the file:
@@
 EESchema Schematic File Version 4
+LIBS:Power supply-cache
 EELAYER 30 0
 EELAYER END
@@
 	1600 1750 1250 1750
 Wire Wire Line
-	1250 1050 2400 1050
+	1250 1050 1600 1050
 Wire Wire Line
 	1250 1750 1250 2750
@@
 $EndComp
 $Comp
-L Timer:NE555P U3
+L Power-supply-rescue:NE555P-Timer U3
 U 1 1 5F239591
 P 3850 4150
@@
 Wire Wire Line
 	7200 3950 7050 3950
+$Comp
+L Device:Fuse F1
+U 1 1 5F1B93A2
+P 1750 1050
+F 0 "F1" V 1553 1050 50  0000 C CNN
+F 1 "3A" V 1644 1050 50  0000 C CNN
+F 2 "Fuse:Fuseholder_Cylinder-5x20mm_Schurter_0031_8201_Horizontal_Open" V 1680 1050 50  0001 C CNN
+F 3 "~" H 1750 1050 50  0001 C CNN
+	1    1750 1050
+	0    1    1    0
+$EndComp
+Wire Wire Line
+	1900 1050 2400 1050
+$Comp
+L Mechanical:Heatsink HS1
+U 1 1 5F1BA977
+P 7000 6350
+F 0 "HS1" H 7142 6471 50  0000 L CNN
+F 1 "Heatsink" H 7142 6380 50  0000 L CNN
+F 2 "ak:HS-160x50" H 7012 6350 50  0001 C CNN
+F 3 "~" H 7012 6350 50  0001 C CNN
+	1    7000 6350
+	1    0    0    -1
+$EndComp
 $EndSCHEMATC

Commit message: PSU
Parts:
- removed J1, J2, J3, J4: Conn_01x01, Connector_Pin:Pin_D1.0mm_L10.0mm, symbol Connector_Generic:Conn_01x01
- added C14: 100nF, Capacitor_THT:C_Disc_D5.0mm_W2.5mm_P2.50mm, symbol Device:C_Small
- added H1, H2, H3, H5, H6, H7: MountingHole_Pad, MountingHole:MountingHole_3.2mm_M3_Pad, symbol Mechanical:MountingHole_Pad
- added H10, H11: MountingHole_Pad, MountingHole:MountingHole_4.3mm_M4_Pad, symbol Mechanical:MountingHole_Pad
- added H12: MountingHole_Pad, MountingHole:MountingHole_5.3mm_M5_Pad, symbol Mechanical:MountingHole_Pad
- added J1: Screw_Terminal_01x04, TerminalBlock_RND:TerminalBlock_RND_205-00003_1x04_P5.00mm_Horizontal, symbol Connector:Screw_Terminal_01x04
- D3, D5, D9: footprint Diode_THT:D_DO-35_SOD27_P7.62mm_Horizontal -> Diode_THT:D_DO-35_SOD27_P10.16mm_Horizontal
- D8: renamed from D7; footprint Diode_THT:D_DO-35_SOD27_P7.62mm_Horizontal -> Diode_THT:D_DO-35_SOD27_P10.16mm_Horizontal
- J2: renamed from J5; footprint Connector_PinHeader_2.54mm:PinHeader_1x04_P2.54mm_Vertical -> Connector_Molex:Molex_KK-396_A-41791-0004_1x04_P3.96mm_Vertical
- renumbered D8 to D7, R4 to R3, R5 to R4, R3 to R5
Connections:
- net +12V: now also J2.4 (Pin_4), K1.A2, C14.1; no longer J2.1 (Pin_1), K1.A1
- net +5V: now also J2.1 (Pin_1); no longer J2.2 (Pin_2)
- net GND: now also J2.2 (Pin_2), C14.2; no longer J2.4 (Pin_4)
- net at D2.2 (~~): now also K1.11, TH1.1; no longer F1.1
- net at F1.2: now also J1.1 (Pin_1), J1.2 (Pin_2)
- net at K1.14, TH1.2: now also J1.3 (Pin_3), J1.4 (Pin_4)
- net at D7.2 (A), Q1.1 (C): now also K1.A1; no longer K1.A2
- new net: D2.3 (~~), F1.1
Other:
- note added: "Heatsink shared between D2, U1 and U2"
- note added: "use AWG#22"
- moved on the sheet: C1, C10, C11, C12, C13, C2, C3, C4, C5, C6, C7, C8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

Commit message: PSU
Connections:
- net at K1.14, TH1.2: now also J1.1 (Pin_1), J1.2 (Pin_2); no longer J1.3 (Pin_3), J1.4 (Pin_4)
- new net: F1.2, J1.3 (Pin_3), J1.4 (Pin_4)
Changed lines of the file:
@@
 EESchema Schematic File Version 4
+LIBS:Power supply-cache
 EELAYER 30 0
 EELAYER END
@@
 L Connector:Screw_Terminal_01x04 J1
 U 1 1 5F1FC0C9
-P 1300 2250
-F 0 "J1" H 1300 2450 50  0000 C CNN
-F 1 "Screw_Terminal_01x04" H 1400 1950 50  0000 C CNN
-F 2 "TerminalBlock_RND:TerminalBlock_RND_205-00003_1x04_P5.00mm_Horizontal" H 1300 2250 50  0001 C CNN
-F 3 "~" H 1300 2250 50  0001 C CNN
-	1    1300 2250
-	-1   0    0    -1
-$EndComp
-Wire Wire Line
+P 1300 2350
+F 0 "J1" H 1300 2550 50  0000 C CNN
+F 1 "Screw_Terminal_01x04" H 1400 2050 50  0000 C CNN
+F 2 "TerminalBlock_RND:TerminalBlock_RND_205-00003_1x04_P5.00mm_Horizontal" H 1300 2350 50  0001 C CNN
+F 3 "~" H 1300 2350 50  0001 C CNN
+	1    1300 2350
+	-1   0    0    1
+$EndComp
+Wire Wire Line
