File: Power_Supply/Power supply.sch (KiCad schematic (older format))
At the start: 49 parts, among them J1 Screw_Terminal_01x04, J2 Conn_01x04, K1 RY611012, Q1 BC548, U1 LM1084-12, U2 LM1084-5, U3 NE555P

Commit message: PSU
Parts:
- added LD1, LD2: LED, LED_THT:LED_D5.0mm, symbol Device:LED
- added LOGO1: Lemonhead, ak:lemonhead, symbol ak:Lemonhead
- added R8: 680R, Resistor_THT:R_Axial_DIN0207_L6.3mm_D2.5mm_P10.16mm_Horizontal, symbol Device:R_Small
- added R9: 220R, Resistor_THT:R_Axial_DIN0207_L6.3mm_D2.5mm_P10.16mm_Horizontal, symbol Device:R_Small
- renumbered D2 to BR1
Connections:
- net +12V: now also LD1.2 (A)
- net +5V: now also LD2.2 (A)
- net GND: now also R8.2, R9.2
- new net: LD1.1 (K), R8.1
- new net: LD2.1 (K), R9.1
- no-connect marks 0 -> 10
Other:
- note removed: "use AWG#22"
- moved on the sheet: BR1, C1, C10, C11, C12, C13, C14, C2, C3, C4, C5, C6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

Commit message: PSU
Parts:
- added R10, R11: 0R, Resistor_THT:R_Axial_DIN0207_L6.3mm_D2.5mm_P10.16mm_Horizontal, symbol Device:R_Small
- added R12, R13: DNP, Resistor_THT:R_Axial_DIN0207_L6.3mm_D2.5mm_P10.16mm_Horizontal, symbol Device:R_Small
- BR1: footprint Diode_THT:Diode_Bridge_Vishay_GBU -> ak:GBJ
Connections:
- net +12V: now also R12.1
- net +5V: now also R13.1
- net GND: now also R10.2, R11.2; no longer U1.1 (ADJ), U2.1 (ADJ)
- new net: R10.1, R12.2, U1.1 (ADJ)
- new net: R11.1, R13.2, U2.1 (ADJ)
Other:
- moved on the sheet: C10, C6, C7, C9, D3, D4, D5, D8, D9, J2, LD1, LD2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

Commit message: PSU
Parts:
- D8: value 5V -> 4V7
- F1: value 3A -> 6A; footprint Fuse:Fuseholder_Cylinder-5x20mm_Schurter_0031_8201_Horizontal_Open -> Fuse:Fuseholder_Cylinder-6.3x32mm_Schurter_0031-8002_Horizontal_Open
- Q2: renamed from D4; value Q_SCR_KAG -> MCR72
- R8: value 680R -> 560R
- R9: value 220R -> 180R
Other:
- note added: "Notes:\n- LD1, LD2 necessary to meet minimum load requirement of U1 and U2.\n- Thyristor crowbar is triggered at approx. 12.7V and 5,4V respectively. \n- U3 switches K1 after approx. 3s."
Changed lines of the file:
@@
 EESchema Schematic File Version 4
-LIBS:Power supply-cache
 EELAYER 30 0
 EELAYER END
@@
 $EndComp
 $Comp
-L Device:Q_SCR_KAG D4
+L Device:Q_SCR_KAG Q2
 U 1 1 5ED58F94
 P 10100 2350
-F 0 "D4" H 10188 2396 50  0000 L CNN
-F 1 "Q_SCR_KAG" H 10188 2305 50  0000 L CNN
+F 0 "Q2" H 10188 2396 50  0000 L CNN
+F 1 "MCR72" H 10188 2305 50  0000 L CNN
 F 2 "Package_TO_SOT_THT:TO-220F-3_Horizontal_TabDown" V 10100 2350 50  0001 C CNN
 F 3 "~" V 10100 2350 50  0001 C CNN
@@
 P 2250 1700
 F 0 "F1" V 2150 1700 50  0000 C CNN
-F 1 "3A" V 2350 1700 50  0000 C CNN
-F 2 "Fuse:Fuseholder_Cylinder-5x20mm_Schurter_0031_8201_Horizontal_Open" V 2180 1700 50  0001 C CNN
+F 1 "6A" V 2350 1700 50  0000 C CNN
+F 2 "Fuse:Fuseholder_Cylinder-6.3x32mm_Schurter_0031-8002_Horizontal_Open" V 2180 1700 50  0001 C CNN
 F 3 "~" H 2250 1700 50  0001 C CNN
 	1    2250 1700
@@
 P 8500 4600
 F 0 "D8" V 8454 4679 50  0000 L CNN
-F 1 "5V" V 8545 4679 50  0000 L CNN
+F 1 "4V7" V 8545 4679 50  0000 L CNN
 F 2 "Diode_THT:D_DO-35_SOD27_P10.16mm_Horizontal" H 8500 4600 50  0001 C CNN
 F 3 "~" H 8500 4600 50  0001 C CNN
@@
 P 8700 4200
 F 0 "R8" H 8759 4246 50  0000 L CNN
-F 1 "680R" H 8759 4155 50  0000 L CNN
+F 1 "560R" H 8759 4155 50  0000 L CNN
 F 2 "Resistor_THT:R_Axial_DIN0207_L6.3mm_D2.5mm_P10.16mm_Horizontal" H 8700 4200 50  0001 C CNN
 F 3 "~" H 8700 4200 50  0001 C CNN
@@
 P 9050 4200
 F 0 "R9" H 9109 4246 50  0000 L CNN
-F 1 "220R" H 9109 4155 50  0000 L CNN
+F 1 "180R" H 9109 4155 50  0000 L CNN
 F 2 "Resistor_THT:R_Axial_DIN0207_L6.3mm_D2.5mm_P10.16mm_Horizontal" H 9050 4200 50  0001 C CNN
 F 3 "~" H 9050 4200 50  0001 C CNN
@@
 	1    0    0    -1
 $EndComp
+Text Notes 6950 5950 0    50   ~ 0
+Notes:\n- LD1, LD2 necessary to meet minimum load requirement of U1 and U2.\n- Thyristor crowbar is triggered at approx. 12.7V and 5,4V respectively. \n- U3 switches K1 after approx. 3s.
 $EndSCHEMATC

Commit message: PSU
Parts:
- R3: value 100k -> 330k
Other:
- note added: "FUCK UP: Circuit starts with relais energized.\nFix: Replace Q1 with PNP"
Changed lines of the file:
@@
 EESchema Schematic File Version 4
+LIBS:Power supply-cache
 EELAYER 30 0
 EELAYER END
@@
 P 4000 4100
 F 0 "R3" H 4059 4146 50  0000 L CNN
-F 1 "100k" H 4059 4055 50  0000 L CNN
+F 1 "330k" H 4059 4055 50  0000 L CNN
 F 2 "Resistor_THT:R_Axial_DIN0207_L6.3mm_D2.5mm_P10.16mm_Horizontal" H 4000 4100 50  0001 C CNN
 F 3 "~" H 4000 4100 50  0001 C CNN
@@
 Text Notes 6950 5950 0    50   ~ 0
 Notes:\n- LD1, LD2 necessary to meet minimum load requirement of U1 and U2.\n- Thyristor crowbar is triggered at approx. 12.7V and 5,4V respectively. \n- U3 switches K1 after approx. 3s.
+Text Notes 1400 5550 0    118  ~ 24
+FUCK UP: Circuit starts with relais energized.\nFix: Replace Q1 with PNP
 $EndSCHEMATC
