File: Power_Supply/Power supply.kicad_pcb (KiCad board)
At the start: 2 copper layers, 140 x 167 mm, 40 parts, among them J1 Conn_01x01, J10 Conn_01x04, J2 Conn_01x01, J3 Conn_01x01, J4 Conn_01x01, J5 Conn_01x01, J6 Conn_01x01, J7 Conn_01x01, J8 Conn_01x01, J9 Conn_01x01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

Commit message: Power supply
Parts:
- moved C6 149.0 mm to (121.0, 48.0), turned to 270 degrees
- moved R3 129.1 mm to (126.0, 54.5)
- moved C9 127.5 mm to (177.5, 47.5), turned to 270 degrees
- moved D1 119.0 mm to (136.0, 48.0), turned to 180 degrees
- moved R1 118.9 mm to (136.2, 51.5), turned to 180 degrees
- moved J10 116.9 mm to (219.0, 58.0)
- moved C5 109.0 mm to (141.0, 48.0), turned to 270 degrees
- moved R5 108.1 mm to (182.0, 51.0)
- moved R7 98.0 mm to (192.2, 54.0), turned to 180 degrees
- moved D6 97.5 mm to (192.5, 47.5), turned to 180 degrees
- moved C8 87.5 mm to (197.5, 47.5), turned to 270 degrees
- moved D2 67.5 mm to (95.0, 85.2), turned to 270 degrees
- moved D4 42.1 mm to (238.0, 76.0), turned to 0 degrees
- moved D8 41.6 mm to (248.5, 70.0)
- moved R8 36.5 mm to (248.5, 76.0)
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
Commit message: psu
Parts:
- removed F1: Fuse, Fuse:Fuseholder_Cylinder-5x20mm_Schurter_0031_8201_Horizontal_Open
- removed J10: Conn_01x04, Connector_PinHeader_2.54mm:PinHeader_1x04_P2.54mm_Vertical
- removed J2, J6, J7, J8, J9: Conn_01x01, Connector_Pin:Pin_D1.0mm_L10.0mm
- removed R8: 470R, Resistor_THT:R_Axial_DIN0207_L6.3mm_D2.5mm_P10.16mm_Horizontal
- removed RV1: S20K275, Varistor:RV_Disc_D21.5mm_W5.4mm_P10mm
- added C11: 10uF, Capacitor_THT:CP_Radial_D5.0mm_P2.00mm, F.Cu at (21.1, -155.9)
- added C12: 100nF, Capacitor_THT:C_Disc_D5.0mm_W2.5mm_P2.50mm, F.Cu at (28.0, -157.9)
- added C13: 100nF, Capacitor_THT:C_Disc_D5.0mm_W2.5mm_P2.50mm, F.Cu at (20.8, -150.6)
- added D9: 1N4148, Diode_THT:D_DO-35_SOD27_P7.62mm_Horizontal, F.Cu at (-2.69, -149.8)
- added K1: RY611012, ak:RY611012, F.Cu at (259.0, 109.0)
- added Q1: BC548, Package_TO_SOT_THT:TO-92_Inline, F.Cu at (27.4, -152.6)
- added TH1: 5R, Varistor:RV_Disc_D21.5mm_W6.1mm_P7.5mm, F.Cu at (247.0, 115.0)
- added U3: NE555P, Package_DIP:DIP-8_W7.62mm, F.Cu at (27.6, -169.6)
- J5: value Conn_01x01 -> Conn_01x04; footprint Connector_Pin:Pin_D1.0mm_L10.0mm -> Connector_PinHeader_2.54mm:PinHeader_1x04_P2.54mm_Vertical
- R1, R3: value ? -> 100R
- R2, R6: value 100R -> 470R
- R4: value 470R -> 100k
- R5: value ? -> 100k
- R7: value ? -> 10k
- U1: value LM1084-ADJ -> LM1084-12
- U2: value LM1084-ADJ -> LM1084-5
- moved J3 246.9 mm to (0.83, -89.9)
- moved J5 244.2 mm to (11.0, -120.4)
- moved C10 229.5 mm to (237.1, -155.2)
- moved C7 229.5 mm to (237.1, -164.7)
- moved D3 229.5 mm to (231.7, -170.2)
- moved D4 229.5 mm to (213.6, -152.2)
- moved D5 229.5 mm to (224.1, -161.2)
- moved D7 229.5 mm to (231.7, -149.2)
- moved D8 229.5 mm to (224.1, -158.2)
- moved R2 229.5 mm to (234.3, -164.2)
- moved R4 229.5 mm to (224.1, -167.2)
- moved R6 229.5 mm to (234.3, -155.2)
- moved J1 219.7 mm to (-1.13, -95.5)
- moved J4 219.7 mm to (3.87, -95.5)
- moved C5 197.9 mm to (236.0, -125.6)
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Connections:
- net Net-(C1-Pad1) renamed VDC
- D8 pad 1: Net-(D4-Pad3) -> +12V
- D8 pad 2: Net-(C10-Pad1) -> Net-(D8-Pad2)
- J3 pad 1: Net-(F1-Pad1) -> Net-(J3-Pad1)
- J4 pad 1: Net-(D2-Pad2) -> Net-(J3-Pad1)
- J5 pad 1: Net-(D2-Pad3) -> +12V
- R1 pad 1: +12V -> Net-(C7-Pad1)
- R1 pad 2: Net-(R1-Pad2) -> Net-(D3-Pad2)
- R2 pad 1: Net-(C7-Pad1) -> Net-(D3-Pad2)
- R2 pad 2: Net-(D3-Pad2) -> GND
- R3 pad 1: Net-(R1-Pad2) -> Net-(C10-Pad1)
- R3 pad 2: GND -> Net-(D7-Pad2)
- R4 pad 1: Net-(D3-Pad2) -> +12V
- R4 pad 2: GND -> Net-(C11-Pad1)
- R5 pad 1: +5V -> +12V
- R5 pad 2: Net-(R5-Pad2) -> Net-(C13-Pad1)
- R6 pad 1: Net-(C10-Pad1) -> Net-(D7-Pad2)
- R6 pad 2: Net-(D7-Pad2) -> GND
- R7 pad 1: Net-(R5-Pad2) -> Net-(R7-Pad1)
- R7 pad 2: GND -> Net-(Q1-Pad2)
- U1 pad 1: Net-(R1-Pad2) -> GND
- U2 pad 1: Net-(R5-Pad2) -> GND
Other:
- board size 140 x 167 mm -> 190.2 x 185.3 mm

Commit message: PSU
Parts:
- added F1: 3A, Fuse:Fuseholder_Cylinder-5x20mm_Schurter_0031_8201_Horizontal_Open, F.Cu at (255.9, 143.3)
- added HS1: Heatsink, ak:HS-160x50, F.Cu at (38.0, 109.0)
- added J2: Conn_01x01, Connector_Pin:Pin_D1.0mm_L10.0mm, F.Cu at (276.6, 181.5)
- moved C12 442.0 mm to (321.2, 172.8)
- moved Q1 439.3 mm to (314.5, 179.9)
- moved C13 398.3 mm to (238.5, 182.9)
- moved J5 396.4 mm to (272.2, 177.8)
- moved J1 395.1 mm to (276.6, 185.6)
- moved D9 393.2 mm to (224.8, 171.0)
- moved J3 384.1 mm to (276.6, 177.4), turned to 0 degrees
- moved C11 383.6 mm to (248.0, 153.4)
- moved U3 377.5 mm to (224.8, 152.2)
- moved J4 357.9 mm to (242.6, 171.2)
- moved R4 352.9 mm to (294.2, 178.7)
- moved D4 343.7 mm to (284.2, 184.2)
- moved R2 342.7 mm to (307.5, 170.6), turned to 0 degrees
- moved D3 337.7 mm to (224.8, 167.4), turned to 0 degrees
- moved R6 331.2 mm to (294.2, 170.6), turned to 0 degrees
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Connections:
- J1 pad 1: Net-(D2-Pad2) -> Net-(F1-Pad2)
- K1 pad 12: Net-(K1-Pad12) -> (no net)
Other:
- board size 190.2 x 185.3 mm -> 180.7 x 180.7 mm

Commit message: PSU
Parts:
- removed J3, J4: Conn_01x01, Connector_Pin:Pin_D1.0mm_L10.0mm
- removed J5: Conn_01x04, Connector_PinHeader_2.54mm:PinHeader_1x04_P2.54mm_Vertical
- removed the R5 at (307.5, 174.6)
- added C14: 100nF, Capacitor_THT:C_Disc_D5.0mm_W2.5mm_P2.50mm, F.Cu at (147.0, 192.0)
- added H1: MountingHole_Pad, MountingHole:MountingHole_3.2mm_M3_Pad, F.Cu at (32.6, 257.0)
- added H10: MountingHole_Pad, MountingHole:MountingHole_4.3mm_M4_Pad, F.Cu at (78.0, 104.0)
- added H11: MountingHole_Pad, MountingHole:MountingHole_4.3mm_M4_Pad, F.Cu at (158.0, 104.0)
- added H12: MountingHole_Pad, MountingHole:MountingHole_5.3mm_M5_Pad, F.Cu at (77.0, 210.2)
- added H2: MountingHole_Pad, MountingHole:MountingHole_3.2mm_M3_Pad, F.Cu at (121.5, 257.0)
- added H3: MountingHole_Pad, MountingHole:MountingHole_3.2mm_M3_Pad, F.Cu at (188.1, 257.0)
- added H5: MountingHole_Pad, MountingHole:MountingHole_3.2mm_M3_Pad, F.Cu at (188.1, 133.3)
- added H6: MountingHole_Pad, MountingHole:MountingHole_3.2mm_M3_Pad, F.Cu at (121.5, 133.3)
- added H7: MountingHole_Pad, MountingHole:MountingHole_3.2mm_M3_Pad, F.Cu at (32.6, 133.3)
- added R3: 100k, Resistor_THT:R_Axial_DIN0207_L6.3mm_D2.5mm_P10.16mm_Horizontal, F.Cu at (156.2, 215.5)
- D3, D5, D9: footprint Diode_THT:D_DO-35_SOD27_P7.62mm_Horizontal -> Diode_THT:D_DO-35_SOD27_P10.16mm_Horizontal
- D8: renamed from D7; footprint Diode_THT:D_DO-35_SOD27_P7.62mm_Horizontal -> Diode_THT:D_DO-35_SOD27_P10.16mm_Horizontal
- J1: value Conn_01x01 -> Screw_Terminal_01x04; footprint Connector_Pin:Pin_D1.0mm_L10.0mm -> TerminalBlock_RND:TerminalBlock_RND_205-00003_1x04_P5.00mm_Horizontal
- J2: value Conn_01x01 -> Conn_01x04; footprint Connector_Pin:Pin_D1.0mm_L10.0mm -> Connector_Molex:Molex_KK-396_A-41791-0004_1x04_P3.96mm_Vertical
- moved D6 236.3 mm to (63.5, 116.5), turned to 180 degrees
- moved R5 217.7 mm to (86.0, 118.8), turned to 270 degrees
- moved R6 215.2 mm to (83.0, 129.0), turned to 90 degrees
- moved C6 214.2 mm to (113.5, 122.0)
- moved R2 213.4 mm to (98.1, 129.0), turned to 90 degrees
- moved C9 199.9 mm to (53.5, 122.0)
- moved C3 198.9 mm to (146.0, 142.0), turned to 180 degrees
- moved C5 193.6 mm to (123.5, 122.0), turned to 180 degrees
- moved D1 191.5 mm to (123.5, 116.5), turned to 180 degrees
- moved C8 188.7 mm to (63.5, 122.0), turned to 180 degrees
- moved U2 187.9 mm to (55.5, 112.5)
- moved D4 183.2 mm to (105.5, 143.5), turned to 270 degrees
- moved C4 172.4 mm to (146.0, 170.0), turned to 180 degrees
- moved C12 167.3 mm to (155.0, 192.0), turned to 180 degrees
- moved Q1 163.9 mm to (155.5, 219.5), turned to 180 degrees
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- renumbered D8 to D7, R3 to R5
Connections:
- D7 pad 2: Net-(D8-Pad2) (its old number) -> Net-(D7-Pad2)
- F1 pad 1: Net-(D2-Pad2) -> Net-(D2-Pad3)
- J2 pad 1: Net-(F1-Pad2) -> +5V
- K1 pad 11: Net-(D2-Pad3) -> Net-(D2-Pad2)
- K1 pad 12: (no net) -> Net-(K1-Pad12)
- K1 pad 14: Net-(J3-Pad1) -> Net-(J1-Pad3)
- K1 pad A1: +12V -> Net-(D7-Pad2)
- K1 pad A2: Net-(D8-Pad2) (its old number) -> +12V
- Q1 pad 1: Net-(D8-Pad2) (its old number) -> Net-(D7-Pad2)
- R4 pad 2: Net-(C11-Pad1) -> Net-(C13-Pad1)
- TH1 pad 1: Net-(D2-Pad3) -> Net-(D2-Pad2)
- TH1 pad 2: Net-(J3-Pad1) -> Net-(J1-Pad3)
Routing:
- net +12V: track 0.00 -> 332.4 mm
- net +5V: track 0.00 -> 230.7 mm
- net Net-(D2-Pad2): track 0.00 -> 144.6 mm
- net Net-(D2-Pad3): track 0.00 -> 116.6 mm
- net VDC: track 0.00 -> 81.4 mm
- net Net-(J1-Pad3): track 0.00 -> 71.1 mm
- net Net-(F1-Pad2): track 0.00 -> 36.2 mm
- net Net-(C11-Pad1): track 0.00 -> 33.9 mm
- net Net-(D4-Pad3): track 0.00 -> 30.8 mm
- net Net-(D7-Pad2): track 0.00 -> 28.3 mm
- net Net-(R7-Pad1): track 0.00 -> 14.7 mm
- net Net-(C13-Pad1): track 0.00 -> 8.55 mm
- net Net-(Q1-Pad2): track 0.00 -> 7.80 mm
- net Net-(D8-Pad2): track 0.00 -> 6.00 mm
- net Net-(D3-Pad2): track 0.00 -> 6.00 mm
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- added copper zone on B.Cu, net GND
- added copper zone on F.Cu, net VDC
Other:
- outline, holes or cut-outs redrawn

Commit message: PSU
Parts:
- moved D4 8.38 mm to (113.5, 146.0), turned to 90 degrees
- moved TH1 7.57 mm to (168.0, 214.0)
- moved C1 6.00 mm to (158.0, 142.0)
- moved C2 6.00 mm to (158.0, 170.0)
- moved J2 6.00 mm to (133.6, 251.0)
- moved C3 4.00 mm to (142.0, 142.0)
- moved C4 4.00 mm to (142.0, 170.0)
- moved F1 0.75 mm to (191.0, 218.8)
Connections:
- H1 pad 1: Net-(H1-Pad1) -> (no net)
- H10 pad 1: Net-(H10-Pad1) -> (no net)
- H11 pad 1: Net-(H11-Pad1) -> (no net)
- H12 pad 1: Net-(H12-Pad1) -> (no net)
- H2 pad 1: Net-(H2-Pad1) -> (no net)
- H3 pad 1: Net-(H3-Pad1) -> (no net)
- H5 pad 1: Net-(H5-Pad1) -> (no net)
- H6 pad 1: Net-(H6-Pad1) -> (no net)
- H7 pad 1: Net-(H7-Pad1) -> (no net)
- J1 pad 1: Net-(F1-Pad2) -> Net-(J1-Pad1)
- J1 pad 2: Net-(F1-Pad2) -> Net-(J1-Pad1)
- J1 pad 3: Net-(J1-Pad3) -> Net-(F1-Pad2)
- J1 pad 4: Net-(J1-Pad3) -> Net-(F1-Pad2)
- K1 pad 12: Net-(K1-Pad12) -> (no net)
- K1 pad 14: Net-(J1-Pad3) -> Net-(J1-Pad1)
- TH1 pad 2: Net-(J1-Pad3) -> Net-(J1-Pad1)
Routing:
- net Net-(J1-Pad3): track 71.1 -> 0.00 mm
- net Net-(J1-Pad1): track 0.00 -> 68.6 mm
- net Net-(F1-Pad2): track 36.2 -> 67.6 mm
- net Net-(D2-Pad2): track 144.6 -> 172.9 mm
- net Net-(D2-Pad3): track 116.6 -> 136.9 mm
- net VDC: track 81.4 -> 69.4 mm
- net +12V: track 332.4 -> 342.8 mm
- net +5V: track 230.7 -> 224.8 mm
- net Net-(D4-Pad3): track 30.8 -> 32.0 mm
Other:
- outline, holes or cut-outs redrawn

Commit message: PSU
Parts:
- added LD1: LED, LED_THT:LED_D5.0mm, F.Cu at (65.0, 132.5)
- added LD2: LED, LED_THT:LED_D5.0mm, F.Cu at (59.5, 132.5)
- added LOGO1: Lemonhead, ak:lemonhead, F.Cu at (137.0, 119.0)
- added R8: 680R, Resistor_THT:R_Axial_DIN0207_L6.3mm_D2.5mm_P10.16mm_Horizontal, F.Cu at (65.0, 137.5)
- added R9: 220R, Resistor_THT:R_Axial_DIN0207_L6.3mm_D2.5mm_P10.16mm_Horizontal, F.Cu at (59.5, 137.5)
- added REF**: KiCad-Logo2_8mm_SilkScreen, Symbol:KiCad-Logo2_8mm_SilkScreen, F.Cu at (144.0, 271.5)
- added REF**: OSHW-Logo2_14.6x12mm_SilkScreen, Symbol:OSHW-Logo2_14.6x12mm_SilkScreen, F.Cu at (124.0, 273.5)
- moved H10 2.50 mm to (80.5, 104.0)
- moved H11 2.50 mm to (160.5, 104.0)
- moved HS1 2.50 mm to (40.5, 109.0)
- renumbered D2 to BR1
Connections:
- H1 pad 1: (no net) -> Net-(H1-Pad1)
- H10 pad 1: (no net) -> Net-(H10-Pad1)
- H11 pad 1: (no net) -> Net-(H11-Pad1)
- H12 pad 1: (no net) -> Net-(H12-Pad1)
- H2 pad 1: (no net) -> Net-(H2-Pad1)
- H3 pad 1: (no net) -> Net-(H3-Pad1)
- H5 pad 1: (no net) -> Net-(H5-Pad1)
- H6 pad 1: (no net) -> Net-(H6-Pad1)
- H7 pad 1: (no net) -> Net-(H7-Pad1)
- K1 pad 12: (no net) -> Net-(K1-Pad12)
Routing:
- net +12V: track 342.8 -> 349.8 mm
- net +5V: track 224.8 -> 230.4 mm
- net Net-(LD2-Pad1): track 0.00 -> 5.00 mm
- net Net-(LD1-Pad1): track 0.00 -> 5.00 mm
- net Net-(F1-Pad2): track 67.6 -> 65.1 mm
- net VDC: track 69.4 -> 71.5 mm
- net Net-(D4-Pad3): track 32.0 -> 32.9 mm
Other:
- outline, holes or cut-outs redrawn
- board text added: "+5V GND GND +12V"
- board text added: "12V"
- board text added: "12V AC IN"
- board text added: "12V/5V Linear Power Supply for 7-Segment RGB Clock Rev. A - 08 / 2020"
- board text added: "5V"
- board text added: "DC OUT"
- board text added: "rot blau gelb grün"

Commit message: PSU
Parts:
- removed REF**: KiCad-Logo2_8mm_SilkScreen, Symbol:KiCad-Logo2_8mm_SilkScreen
- removed REF**: OSHW-Logo2_14.6x12mm_SilkScreen, Symbol:OSHW-Logo2_14.6x12mm_SilkScreen
- added R10: 0R, Resistor_THT:R_Axial_DIN0207_L6.3mm_D2.5mm_P10.16mm_Horizontal, F.Cu at (106.5, 112.5)
- added R11: 0R, Resistor_THT:R_Axial_DIN0207_L6.3mm_D2.5mm_P10.16mm_Horizontal, F.Cu at (46.5, 112.5)
- added R12: DNP, Resistor_THT:R_Axial_DIN0207_L6.3mm_D2.5mm_P10.16mm_Horizontal, F.Cu at (109.5, 122.7)
- added R13: DNP, Resistor_THT:R_Axial_DIN0207_L6.3mm_D2.5mm_P10.16mm_Horizontal, F.Cu at (49.5, 122.7)
- BR1: footprint Diode_THT:Diode_Bridge_Vishay_GBU -> ak:GBJ
- moved BR1 8.43 mm to (162.2, 112.2)
Connections:
- H1 pad 1: Net-(H1-Pad1) -> (no net)
- H10 pad 1: Net-(H10-Pad1) -> (no net)
- H11 pad 1: Net-(H11-Pad1) -> (no net)
- H12 pad 1: Net-(H12-Pad1) -> (no net)
- H2 pad 1: Net-(H2-Pad1) -> (no net)
- H3 pad 1: Net-(H3-Pad1) -> (no net)
- H5 pad 1: Net-(H5-Pad1) -> (no net)
- H6 pad 1: Net-(H6-Pad1) -> (no net)
- H7 pad 1: Net-(H7-Pad1) -> (no net)
- K1 pad 12: Net-(K1-Pad12) -> (no net)
- U1 pad 1: GND -> Net-(R10-Pad1)
- U2 pad 1: GND -> Net-(R11-Pad1)
Routing:
- net Net-(R11-Pad1): track 0.00 -> 8.96 mm
- net Net-(R10-Pad1): track 0.00 -> 8.96 mm
- net +12V: track 349.8 -> 356.9 mm
- net Net-(BR1-Pad3): track 136.9 -> 132.5 mm
- net +5V: track 230.4 -> 234.7 mm

Commit message: PSU
Parts:
- moved H7 30.0 mm to (32.6, 163.3)
Other:
- outline, holes or cut-outs redrawn
Changed lines of the file:
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@@
   )
   (setup
-    (last_trace_width 0.5)
+    (last_trace_width 0.25)
     (user_trace_width 0.5)
     (user_trace_width 1)
@@
     (add_net "Net-(D8-Pad2)")
     (add_net "Net-(F1-Pad2)")
-    (add_net "Net-(H1-Pad1)")
-    (add_net "Net-(H10-Pad1)")
-    (add_net "Net-(H11-Pad1)")
-    (add_net "Net-(H12-Pad1)")
-    (add_net "Net-(H2-Pad1)")
-    (add_net "Net-(H3-Pad1)")
-    (add_net "Net-(H5-Pad1)")
-    (add_net "Net-(H6-Pad1)")
-    (add_net "Net-(H7-Pad1)")
     (add_net "Net-(J1-Pad1)")
-    (add_net "Net-(K1-Pad12)")
     (add_net "Net-(LD1-Pad1)")
     (add_net "Net-(LD2-Pad1)")
@@
   )
   (module MountingHole:MountingHole_3.2mm_M3_Pad locked (layer F.Cu)
-    (at 32.56 133.3)
+    (at 32.56 163.3)
     (descr "Mounting Hole 3.2mm, M3")
     (tags "mounting hole 3.2mm m3")
@@
   (gr_circle (center 188.14 103.300001) (end 190.64 103.300001) (layer B.SilkS) (width 0.2))
   (gr_circle (center 188.14 193.300001) (end 190.64 193.300001) (layer B.SilkS) (width 0.2))
-  (gr_circle (center 32.56 163.3) (end 35.06 163.3) (layer B.SilkS) (width 0.2))
+  (gr_circle (center 32.56 133.3) (end 35.06 133.3) (layer B.SilkS) (width 0.2))
   (gr_circle (center 188.14 163.300001) (end 190.64 163.300001) (layer B.SilkS) (width 0.2))
   (gr_circle (center 121.46 223.3) (end 123.96 223.3) (layer B.SilkS) (width 0.2))
@@
   (gr_circle (center 32.56 223.3) (end 35.06 223.3) (layer B.SilkS) (width 0.2))
   (gr_circle (center 121.46 163.3) (end 123.96 163.3) (layer B.SilkS) (width 0.2))
-  (gr_arc (start 28 212.3) (end 28 213.3) (angle -90) (layer Edge.Cuts) (width 0.05))
-  (gr_line (start 28 213.3) (end 27 213.3) (layer Edge.Cuts) (width 0.05))
-  (gr_line (start 29 208.3) (end 29 212.3) (layer Edge.Cuts) (width 0.05))
-  (gr_arc (start 27 212.3) (end 26 212.3) (angle -90) (layer Edge.Cuts) (width 0.05))
-  (gr_line (start 26 212.3) (end 26 208.3) (layer Edge.Cuts) (width 0.05))
-  (gr_arc (start 27 208.3) (end 27 207.3) (angle -90) (layer Edge.Cuts) (width 0.05))
-  (gr_line (start 27 207.3) (end 28 207.3) (layer Edge.Cuts) (width 0.05))
-  (gr_arc (start 28 208.3) (end 29 208.3) (angle -90) (layer Edge.Cuts) (width 0.05))
-  (gr_line (start 125 212.15) (end 125 208.15) (layer Edge.Cuts) (width 0.05))
-  (gr_line (start 128 208.15) (end 128 212.15) (layer Edge.Cuts) (width 0.05))
-  (gr_arc (start 127 212.15) (end 127 213.15) (angle -90) (layer Edge.Cuts) (width 0.05))
-  (gr_arc (start 126 212.15) (end 125 212.15) (angle -90) (layer Edge.Cuts) (width 0.05))
-  (gr_line (start 126 207.15) (end 127 207.15) (layer Edge.Cuts) (width 0.05))
-  (gr_line (start 127 213.15) (end 126 213.15) (layer Edge.Cuts) (width 0.05))
-  (gr_arc (start 126 208.15) (end 126 207.15) (angle -90) (layer Edge.Cuts) (width 0.05))
-  (gr_arc (start 127 208.15) (end 128 208.15) (angle -90) (layer Edge.Cuts) (width 0.05))
-  (gr_line (start 67 208.25) (end 67 212.25) (layer Edge.Cuts) (width 0.05))
-  (gr_line (start 64 212.25) (end 64 208.25) (layer Edge.Cuts) (width 0.05))
-  (gr_arc (start 65 208.25) (end 65 207.25) (angle -90) (layer Edge.Cuts) (width 0.05))
-  (gr_arc (start 66 208.25) (end 67 208.25) (angle -90) (layer Edge.Cuts) (width 0.05))
-  (gr_line (start 66 213.25) (end 65 213.25) (layer Edge.Cuts) (width 0.05))
-  (gr_line (start 65 207.25) (end 66 207.25) (layer Edge.Cuts) (width 0.05))
-  (gr_arc (start 66 212.25) (end 66 213.25) (angle -90) (layer Edge.Cuts) (width 0.05))
-  (gr_arc (start 65 212.25) (end 64 212.25) (angle -90) (layer Edge.Cuts) (width 0.05))
-  (gr_line (start 88 207.25) (end 89 207.25) (layer Edge.Cuts) (width 0.05))
-  (gr_line (start 87 212.25) (end 87 208.25) (layer Edge.Cuts) (width 0.05))
-  (gr_line (start 89 213.25) (end 88 213.25) (layer Edge.Cuts) (width 0.05))
-  (gr_line (start 90 208.25) (end 90 212.25) (layer Edge.Cuts) (width 0.05))
-  (gr_arc (start 89 212.25) (end 89 213.25) (angle -90) (layer Edge.Cuts) (width 0.05))
-  (gr_arc (start 88 212.25) (end 87 212.25) (angle -90) (layer Edge.Cuts) (width 0.05))
-  (gr_arc (start 89 208.25) (end 90 208.25) (angle -90) (layer Edge.Cuts) (width 0.05))
-  (gr_arc (start 88 208.25) (end 88 207.25) (angle -90) (layer Edge.Cuts) (width 0.05))
+  (gr_arc (start 30 212.3) (end 30 213.3) (angle -90) (layer Edge.Cuts) (width 0.05))
+  (gr_line (start 30 213.3) (end 29 213.3) (layer Edge.Cuts) (width 0.05))
+  (gr_line (start 31 208.3) (end 31 212.3) (layer Edge.Cuts) (width 0.05))
+  (gr_arc (start 29 212.3) (end 28 212.3) (angle -90) (layer Edge.Cuts) (width 0.05))
+  (gr_line (start 28 212.3) (end 28 208.3) (layer Edge.Cuts) (width 0.05))
+  (gr_arc (start 29 208.3) (end 29 207.3) (angle -90) (layer Edge.Cuts) (width 0.05))
+  (gr_line (start 29 207.3) (end 30 207.3) (layer Edge.Cuts) (width 0.05))
+  (gr_arc (start 30 208.3) (end 31 208.3) (angle -90) (layer Edge.Cuts) (width 0.05))
+  (gr_line (start 123 212.15) (end 123 208.15) (layer Edge.Cuts) (width 0.05))
+  (gr_line (start 126 208.15) (end 126 212.15) (layer Edge.Cuts) (width 0.05))
+  (gr_arc (start 125 212.15) (end 125 213.15) (angle -90) (layer Edge.Cuts) (width 0.05))
+  (gr_arc (start 124 212.15) (end 123 212.15) (angle -90) (layer Edge.Cuts) (width 0.05))
+  (gr_line (start 124 207.15) (end 125 207.15) (layer Edge.Cuts) (width 0.05))
+  (gr_line (start 125 213.15) (end 124 213.15) (layer Edge.Cuts) (width 0.05))
+  (gr_arc (start 124 208.15) (end 124 207.15) (angle -90) (layer Edge.Cuts) (width 0.05))
+  (gr_arc (start 125 208.15) (end 126 208.15) (angle -90) (layer Edge.Cuts) (width 0.05))
+  (gr_line (start 66 208.25) (end 66 212.25) (layer Edge.Cuts) (width 0.05))
+  (gr_line (start 63 212.25) (end 63 208.25) (layer Edge.Cuts) (width 0.05))
+  (gr_arc (start 64 208.25) (end 64 207.25) (angle -90) (layer Edge.Cuts) (width 0.05))
+  (gr_arc (start 65 208.25) (end 66 208.25) (angle -90) (layer Edge.Cuts) (width 0.05))
+  (gr_line (start 65 213.25) (end 64 213.25) (layer Edge.Cuts) (width 0.05))
+  (gr_line (start 64 207.25) (end 65 207.25) (layer Edge.Cuts) (width 0.05))
+  (gr_arc (start 65 212.25) (end 65 213.25) (angle -90) (layer Edge.Cuts) (width 0.05))
+  (gr_arc (start 64 212.25) (end 63 212.25) (angle -90) (layer Edge.Cuts) (width 0.05))
+  (gr_line (start 89 207.25) (end 90 207.25) (layer Edge.Cuts) (width 0.05))
+  (gr_line (start 88 212.25) (end 88 208.25) (layer Edge.Cuts) (width 0.05))
+  (gr_line (start 90 213.25) (end 89 213.25) (layer Edge.Cuts) (width 0.05))
+  (gr_line (start 91 208.25) (end 91 212.25) (layer Edge.Cuts) (width 0.05))
+  (gr_arc (start 90 212.25) (end 90 213.25) (angle -90) (layer Edge.Cuts) (width 0.05))
+  (gr_arc (start 89 212.25) (end 88 212.25) (angle -90) (layer Edge.Cuts) (width 0.05))
+  (gr_arc (start 90 208.25) (end 91 208.25) (angle -90) (layer Edge.Cuts) (width 0.05))
+  (gr_arc (start 89 208.25) (end 89 207.25) (angle -90) (layer Edge.Cuts) (width 0.05))
   (gr_circle (center 77 210.15) (end 92 210.15) (layer F.SilkS) (width 0.5))
-  (gr_circle (center 77 210.15) (end 123 210.15) (layer F.SilkS) (width 0.5))
+  (gr_circle (center 77 210.15) (end 122 210.15) (layer F.SilkS) (width 0.5))
   (gr_line (start 20 99.300001) (end 200.7 99.300001) (layer Edge.Cuts) (width 0.2))
   (gr_line (start 20 280) (end 20 99.300001) (layer Edge.Cuts) (width 0.2))
