File: Power_Supply/Power supply.kicad_pcb (KiCad board)
At the start: 2 copper layers, 180.7 x 180.7 mm, 58 parts, among them J1 Screw_Terminal_01x04, J2 Conn_01x04, K1 RY611012, Q1 BC548, U1 LM1084-12, U2 LM1084-5, U3 NE555P

Commit message: PSU
Parts:
- D8: value 5V -> 4V7
- F1: value 3A -> 6A; footprint Fuse:Fuseholder_Cylinder-5x20mm_Schurter_0031_8201_Horizontal_Open -> Fuse:Fuseholder_Cylinder-6.3x32mm_Schurter_0031-8002_Horizontal_Open
- Q2: renamed from D4; value Q_SCR_KAG -> MCR72
- R8: value 680R -> 560R
- R9: value 220R -> 180R
- moved F1 11.9 mm to (193.0, 207.0)
Connections:
- H1 pad 1: (no net) -> Net-(H1-Pad1)
- H10 pad 1: (no net) -> Net-(H10-Pad1)
- H11 pad 1: (no net) -> Net-(H11-Pad1)
- H12 pad 1: (no net) -> Net-(H12-Pad1)
- H2 pad 1: (no net) -> Net-(H2-Pad1)
- H3 pad 1: (no net) -> Net-(H3-Pad1)
- H5 pad 1: (no net) -> Net-(H5-Pad1)
- H6 pad 1: (no net) -> Net-(H6-Pad1)
- H7 pad 1: (no net) -> Net-(H7-Pad1)
- K1 pad 12: (no net) -> Net-(K1-Pad12)
Routing:
- net Net-(BR1-Pad3): track 132.5 -> 119.9 mm
- net Net-(F1-Pad2): track 65.1 -> 61.0 mm
- net Net-(BR1-Pad2): track 173.0 -> 176.0 mm

Commit message: PSU
Parts:
- J2: footprint Connector_Molex:Molex_KK-396_A-41791-0004_1x04_P3.96mm_Vertical -> ak:Molex_KK-396_A-41791-0004_1x04_P3.96mm_Vertical
- R3: value 100k -> 330k
