File: Controller Rev. B/Controller.kicad_pcb (KiCad board)
At the start: 2 copper layers, 213 x 24 mm, 94 parts, among them J1 DATA, J2 15V, J3 ICSP, J4 DC OUT, J5 5V, J6 5V AUX, J7 USB, Q1 SI4435FDY, Q2 SI4435FDY, Q3 SQ2309ES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

Commit message: Update
Parts:
- F3: value 0.5A -> Polyfuse 500mA
- F4: value 500mA -> Polyfuse 500mA
- J1: value DATA -> Conn_02x04_Top_Bottom
- J3: value ICSP -> Conn_02x03_Top_Bottom
- J4: value DC OUT -> Conn_02x04_Top_Bottom
- J6: value 5V AUX -> Conn_01x02
- J7: value USB -> USB_A
- JP1: value 5V PASSTHRU -> Jumper
- LD1, LD2: value blue -> LED blue
- LD3, LD5: value orange -> LED
- LD4, LD6: value green -> LED
- LD7: value red -> LED
- U2: value ATmega328P -> ATmega328P-AU
