File: Controller Rev. B/Controller.sch (KiCad schematic (older format))
At the start: 94 parts, among them J1 DATA, J2 15V, J3 ICSP, J4 DC OUT, J5 5V, J6 5V AUX, J7 USB, Q1 SI4435FDY, Q2 SI4435FDY, Q3 SQ2309ES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

Commit message: Update
Parts:
- removed H1, H2: Mounting Hole, MountingHole:MountingHole_3.2mm_M3_Pad_Via, symbol Mechanical:MountingHole_Pad
- removed TP1: RTC_1PPS, TestPoint:TestPoint_Pad_D2.0mm, symbol Connector:TestPoint_Alt
- removed TP10: TLC_LAT, TestPoint:TestPoint_Pad_D2.0mm, symbol Connector:TestPoint_Alt
- removed TP11: TLC_BLANK, TestPoint:TestPoint_Pad_D2.0mm, symbol Connector:TestPoint_Alt
- removed TP12: +BATT, TestPoint:TestPoint_Pad_D2.0mm, symbol Connector:TestPoint_Alt
- removed TP13: VBUS, TestPoint:TestPoint_Pad_D2.0mm, symbol Connector:TestPoint_Alt
- removed TP16: +15V, TestPoint:TestPoint_Pad_D2.0mm, symbol Connector:TestPoint_Alt
- removed TP2, TP4: GND, TestPoint:TestPoint_Loop_D2.60mm_Drill1.6mm_Beaded, symbol Connector:TestPoint_Alt
- removed TP3: RTC_32K, TestPoint:TestPoint_Pad_D2.0mm, symbol Connector:TestPoint_Alt
- removed TP5: PD_OUT, TestPoint:TestPoint_Pad_D2.0mm, symbol Connector:TestPoint_Alt
- removed TP7: TLC_SDA, TestPoint:TestPoint_Pad_D2.0mm, symbol Connector:TestPoint_Alt
- removed TP9: TLC_SCL, TestPoint:TestPoint_Pad_D2.0mm, symbol Connector:TestPoint_Alt
- C1, C2: Manufacturer (none) -> EMVE250ADA331MJA0G; Mouser 700-DS3231M+TRL -> 661-EMVE250ADA331MJA; RS (none) -> 569-287
- C10, C12, C13, C15, C16, C18, C20, C21, C22, C24, C27, C7, C8: Manufacturer (none) -> 1812L050PR; RS (none) -> 787-4218
- C11, C9: Manufacturer (none) -> EEE-FK1K4R7P; Mouser 700-DS3231M+TRL -> 667-EEE-FK1K4R7P; RS (none) -> 715-1433
- C14, C17, C19, C6: Manufacturer (none) -> 885012206089; RS (none) -> 839-2950
- C23: Manufacturer (none) -> TMK107B7105MA-T; RS (none) -> 723-4972
- C25: value 100nF -> ??; Mouser 576-1812L050PR -> (none)
- C26: Manufacturer (none) -> FC0H105ZFTBR44-SS; RS (none) -> 135-6149
- C3: Manufacturer (none) -> 885012207092; RS (none) -> 181-4072
- C4, C5: Manufacturer (none) -> UUR1A101MCL1GS; RS (none) -> 715-1174
- D1: renamed from D9; value SS1P3L -> MBR130; Manufacturer (none) -> MBR130T1G; Mouser (none) -> 863-MBR130T1G; RS (none) -> 688-0492
- D2: renamed from D3; value SS1P3L -> MBR130; Manufacturer (none) -> MBR130T1G; Mouser (none) -> 863-MBR130T1G; RS (none) -> 688-0492
- F1: Manufacturer (none) -> 0154004.DRT; RS (none) -> 219-6125
- F2: Manufacturer (none) -> 0154001.DR; RS (none) -> 219-6096
- F3, F4: Manufacturer (none) -> 1812L050PR; RS (none) -> 1812L050PR
- J1: value DATA -> Conn_02x04_Top_Bottom; Label (none) -> Data; Manufacturer (none) -> M20-8890845
- J2: footprint Connector_JST:JST_XH_B2B-XH-A_1x02_P2.50mm_Vertical -> Connectors_JST:JST_XH_B03B-XH-A_03x2.50mm_Straight; symbol Connector_Generic:Conn_01x02 -> Connector_Generic:Conn_01x03; Digikey (none) -> 455-2248-ND
- J3: value ICSP -> Conn_02x03_Top_Bottom; Digikey (none) -> 732-5394-ND; Label (none) -> ICSP
- J4: value DC OUT -> Conn_02x04_Top_Bottom; Label (none) -> DC out; Manufacturer (none) -> M20-8890845
- J5: Digikey (none) -> 455-2247-ND
- J6: value 5V AUX -> Conn_01x02; Digikey (none) -> 455-2247-ND; Label (none) -> 5V aux
- J7: value USB -> USB_A; Manufacturer (none) -> 61729-0011BLF; Mouser (none) -> 649-61729-0011BLF; RS (none) -> 172-5271
- JP1: value 5V PASSTHRU -> Jumper; Digikey (none) -> S1012EC-02-ND; Label (none) -> 5V passthrough
- L1, L2, L3: Manufacturer (none) -> LBR2012T100K; RS (none) -> 724-2728
- LD1: renamed from D1; Manufacturer (none) -> LTST-C193TBKT-5A; Mouser (none) -> 859-LTSTC193TBKT5A; RS (none) -> 692-1051
- LD2: renamed from D2; Manufacturer (none) -> LTST-C193TBKT-5A; Mouser (none) -> 859-LTSTC193TBKT5A; RS (none) -> 692-1051
- LD3: renamed from D4; value LED orange -> LED; Label (none) -> Orange; Mouser (none) -> 859-LTST-C191KFKT
- LD4: renamed from D5; value LED green -> LED; Label (none) -> Green; Mouser (none) -> 859-LTST-C190KGKT
- LD5: renamed from D6; value LED orange -> LED; Label (none) -> Orange; Mouser (none) -> 859-LTST-C191KFKT
- LD6: renamed from D7; value LED green -> LED; Label (none) -> Green; Mouser (none) -> 859-LTST-C190KGKT
- LD7: renamed from D8; value LED red -> LED; Label (none) -> Red; Mouser (none) -> 859-LTST-C190KRKT
- PD1: Manufacturer (none) -> SFH 2440; RS (none) -> 124-3361
- Q1, Q2: Manufacturer (none) -> SI4435FDY-T1-GE3; Mouser (none) -> 78-SI4435FDY-T1-GE3; RS (none) -> 710-3339
- Q3: Manufacturer (none) -> SQ2309ES-T1_GE3; Mouser (none) -> 781-SQ2309ES-T1_GE3; RS (none) -> 180-7990
- R1, R13, R2, R3, R4, R5, R6, R7: Manufacturer (none) -> RN73H1JT1001F100; Mouser (none) -> 660-RN73H1JT1001F100; RS (none) -> 213-2266
- R11, R12: Manufacturer (none) -> RN73H1JTD1002F50; Mouser (none) -> 660-RN73H1JTD1002F50; RS (none) -> 678-9667
- R14: Manufacturer (none) -> RN73H1JT1000F100; Mouser (none) -> 660-RN73H1JT1000F100; RS (none) -> 740-8798
- R16, R17, R8, R9: Manufacturer (none) -> RN73H1JT4701F100; Mouser (none) -> 660-RN73H1JT4701F100; RS (none) -> 679-0484
- U1: Manufacturer (none) -> FT232RL; RS (none) -> 406-580
- U2: Manufacturer (none) -> ATMEGA328P-AU; Mouser (none) -> 556-ATMEGA328P-AU; RS (none) -> 131-0271
- U3: Manufacturer (none) -> DS3231M+TRL; RS (none) -> 191-3543
- U4: Manufacturer (none) -> SN74AHC1G14DBVR; Mouser (none) -> 595-SN74AHC1G14DBVR; RS (none) -> 526-381
- U5: symbol ak:LMV301 -> Controller-rescue:LMV301-ak; Manufacturer (none) -> LMV301MGX/NOPB
- Y1: Manufacturer (none) -> CSTNE16M0V53Z000R; RS (none) -> 702-7305
Connections:
- net labels added: Mounting Hole
- wire segments 327 -> 328

Commit message: Update
Parts:
- added TP1: RTC_1PPS, TestPoint:TestPoint_Pad_D2.0mm, symbol Connector:TestPoint_Alt
- added TP10: TLC_LAT, TestPoint:TestPoint_Pad_D2.0mm, symbol Connector:TestPoint_Alt
- added TP11: TLC_BLANK, TestPoint:TestPoint_Pad_D2.0mm, symbol Connector:TestPoint_Alt
- added TP12: +BATT, TestPoint:TestPoint_Pad_D2.0mm, symbol Connector:TestPoint_Alt
- added TP13: VBUS, TestPoint:TestPoint_Pad_D2.0mm, symbol Connector:TestPoint_Alt
- added TP16: +15V, TestPoint:TestPoint_Pad_D2.0mm, symbol Connector:TestPoint_Alt
- added TP2, TP4: GND, TestPoint:TestPoint_Loop_D2.60mm_Drill1.6mm_Beaded, symbol Connector:TestPoint_Alt
- added TP3: RTC_32K, TestPoint:TestPoint_Pad_D2.0mm, symbol Connector:TestPoint_Alt
- added TP5: PD_OUT, TestPoint:TestPoint_Pad_D2.0mm, symbol Connector:TestPoint_Alt
- added TP7: TLC_SDA, TestPoint:TestPoint_Pad_D2.0mm, symbol Connector:TestPoint_Alt
- added TP9: TLC_SCL, TestPoint:TestPoint_Pad_D2.0mm, symbol Connector:TestPoint_Alt
Changed lines of the file:
@@
 $EndComp
 $Comp
-L Connector:TestPoint_Alt #TP16
+L Connector:TestPoint_Alt TP16
 U 1 1 5EA15311
 P 10200 2250
-F 0 "#TP16" V 10200 2650 50  0000 R CNN
+F 0 "TP16" V 10200 2650 50  0000 R CNN
 F 1 "+15V" H 10142 2367 50  0001 R CNN
 F 2 "TestPoint:TestPoint_Pad_D2.0mm" H 10400 2250 50  0001 C CNN
@@
 $EndComp
 $Comp
-L Connector:TestPoint_Alt #TP13
+L Connector:TestPoint_Alt TP13
 U 1 1 5EA2EDBD
 P 10200 2150
-F 0 "#TP13" V 10200 2550 50  0000 R CNN
+F 0 "TP13" V 10200 2550 50  0000 R CNN
 F 1 "VBUS" H 10142 2267 50  0001 R CNN
 F 2 "TestPoint:TestPoint_Pad_D2.0mm" H 10400 2150 50  0001 C CNN
@@
 $EndComp
 $Comp
-L Connector:TestPoint_Alt #TP12
+L Connector:TestPoint_Alt TP12
 U 1 1 5EA2F1A5
 P 10200 2050
-F 0 "#TP12" V 10200 2450 50  0000 R CNN
+F 0 "TP12" V 10200 2450 50  0000 R CNN
 F 1 "+BATT" H 10142 2167 50  0001 R CNN
 F 2 "TestPoint:TestPoint_Pad_D2.0mm" H 10400 2050 50  0001 C CNN
@@
 $EndComp
 $Comp
-L Connector:TestPoint_Alt #TP11
+L Connector:TestPoint_Alt TP11
 U 1 1 5ECA4422
 P 10200 1900
-F 0 "#TP11" V 10200 2300 50  0000 R CNN
+F 0 "TP11" V 10200 2300 50  0000 R CNN
 F 1 "TLC_BLANK" H 10142 2017 50  0001 R CNN
 F 2 "TestPoint:TestPoint_Pad_D2.0mm" H 10400 1900 50  0001 C CNN
@@
 $EndComp
 $Comp
-L Connector:TestPoint_Alt #TP10
+L Connector:TestPoint_Alt TP10
 U 1 1 5EC8ADD5
 P 10200 1800
-F 0 "#TP10" V 10200 2200 50  0000 R CNN
+F 0 "TP10" V 10200 2200 50  0000 R CNN
 F 1 "TLC_LAT" H 10142 1917 50  0001 R CNN
 F 2 "TestPoint:TestPoint_Pad_D2.0mm" H 10400 1800 50  0001 C CNN
@@
 $EndComp
 $Comp
-L Connector:TestPoint_Alt #TP9
+L Connector:TestPoint_Alt TP9
 U 1 1 5EC71932
 P 10200 1700
-F 0 "#TP9" V 10200 2050 50  0000 R CNN
+F 0 "TP9" V 10200 2050 50  0000 R CNN
 F 1 "TLC_SCL" H 10142 1817 50  0001 R CNN
 F 2 "TestPoint:TestPoint_Pad_D2.0mm" H 10400 1700 50  0001 C CNN
@@
 $EndComp
 $Comp
-L Connector:TestPoint_Alt #TP7
+L Connector:TestPoint_Alt TP7
 U 1 1 5EC3E132
 P 10200 1600
-F 0 "#TP7" V 10200 1950 50  0000 R CNN
+F 0 "TP7" V 10200 1950 50  0000 R CNN
 F 1 "TLC_SDA" H 10142 1717 50  0001 R CNN
 F 2 "TestPoint:TestPoint_Pad_D2.0mm" H 10400 1600 50  0001 C CNN
@@
 $EndComp
 $Comp
-L Connector:TestPoint_Alt #TP5
+L Connector:TestPoint_Alt TP5
 U 1 1 5EC25000
 P 10200 1500
-F 0 "#TP5" V 10200 1850 50  0000 R CNN
+F 0 "TP5" V 10200 1850 50  0000 R CNN
 F 1 "PD_OUT" H 10142 1617 50  0001 R CNN
 F 2 "TestPoint:TestPoint_Pad_D2.0mm" H 10400 1500 50  0001 C CNN
@@
 $EndComp
 $Comp
-L Connector:TestPoint_Alt #TP3
+L Connector:TestPoint_Alt TP3
 U 1 1 5EC0C17D
 P 10200 1400
-F 0 "#TP3" V 10200 1750 50  0000 R CNN
+F 0 "TP3" V 10200 1750 50  0000 R CNN
 F 1 "RTC_32K" H 10142 1517 50  0001 R CNN
 F 2 "TestPoint:TestPoint_Pad_D2.0mm" H 10400 1400 50  0001 C CNN
@@
 $EndComp
 $Comp
-L Connector:TestPoint_Alt #TP2
+L Connector:TestPoint_Alt TP2
 U 1 1 5EE4DC32
 P 11000 1300
-F 0 "#TP2" V 11000 1650 50  0000 R CNN
+F 0 "TP2" V 11000 1650 50  0000 R CNN
 F 1 "GND" H 10942 1417 50  0001 R CNN
 F 2 "TestPoint:TestPoint_Loop_D2.60mm_Drill1.6mm_Beaded" H 11200 1300 50  0001 C CNN
@@
 $EndComp
 $Comp
-L Connector:TestPoint_Alt #TP4
+L Connector:TestPoint_Alt TP4
 U 1 1 5EAC13B7
 P 11000 1400
-F 0 "#TP4" V 11000 1750 50  0000 R CNN
+F 0 "TP4" V 11000 1750 50  0000 R CNN
 F 1 "GND" H 10942 1517 50  0001 R CNN
 F 2 "TestPoint:TestPoint_Loop_D2.60mm_Drill1.6mm_Beaded" H 11200 1400 50  0001 C CNN
@@
 $EndComp
 $Comp
-L Connector:TestPoint_Alt #TP1
+L Connector:TestPoint_Alt TP1
 U 1 1 5EBF1B77
 P 10200 1300
-F 0 "#TP1" V 10200 1650 50  0000 R CNN
+F 0 "TP1" V 10200 1650 50  0000 R CNN
 F 1 "RTC_1PPS" H 10142 1417 50  0001 R CNN
 F 2 "TestPoint:TestPoint_Pad_D2.0mm" H 10400 1300 50  0001 C CNN

Commit message: Minor changes
Parts:
- C11, C9: RS 715-1433 -> (none)
Other:
- note added: "Footprint Q1,Q2 too large!"
Changed lines of the file:
@@
 F 4 "667-EEE-FK1K4R7P" H 4550 4250 50  0001 C CNN "Mouser"
 F 5 "EEE-FK1K4R7P" H 4550 4250 50  0001 C CNN "Manufacturer"
-F 6 "715-1433" H 4550 4250 50  0001 C CNN "RS"
+F 6 "" H 4550 4250 50  0001 C CNN "RS"
 	1    4550 4250
 	1    0    0    -1
@@
 $EndComp
 $Comp
-L Device:CP_Small C9
-U 1 1 5D9A4EA0
-P 2450 4250
-F 0 "C9" H 2538 4296 50  0000 L CNN
-F 1 "4u7" H 2538 4205 50  0000 L CNN
-F 2 "Capacitor_SMD:C_Elec_4x5.8" H 2450 4250 50  0001 C CNN
-F 3 "~" H 2450 4250 50  0001 C CNN
-F 4 "667-EEE-FK1K4R7P" H 2450 4250 50  0001 C CNN "Mouser"
-F 5 "EEE-FK1K4R7P" H 2450 4250 50  0001 C CNN "Manufacturer"
-F 6 "715-1433" H 2450 4250 50  0001 C CNN "RS"
-	1    2450 4250
-	1    0    0    -1
-$EndComp
-$Comp
 L Device:R_Small R14
 U 1 1 5DF1C644
@@
 	0    1    -1   0
 $EndComp
+$Comp
+L Device:CP_Small C9
+U 1 1 5D9A4EA0
+P 2450 4250
+F 0 "C9" H 2538 4296 50  0000 L CNN
+F 1 "4u7" H 2538 4205 50  0000 L CNN
+F 2 "Capacitor_SMD:C_Elec_4x5.8" H 2450 4250 50  0001 C CNN
+F 3 "~" H 2450 4250 50  0001 C CNN
+F 4 "667-EEE-FK1K4R7P" H 2450 4250 50  0001 C CNN "Mouser"
+F 5 "EEE-FK1K4R7P" H 2450 4250 50  0001 C CNN "Manufacturer"
+F 6 "" H 2450 4250 50  0001 C CNN "RS"
+	1    2450 4250
+	1    0    0    -1
+$EndComp
+Text Notes 4800 3000 0    79   ~ 16
+Footprint Q1,Q2 too large!
 $EndSCHEMATC
