File: Digit/Digit.sch (KiCad schematic (older format))
At the start: 106 parts, among them J1 Power In, J2 Power out, J3 Signal in, J4 Signal out, U1 TLC5952, U2 TLC5952, U3 74LS244

Commit message: Minor changes. BOM
Parts:
- J1: value Power In -> DC IN
- J2: value Power out -> DC OUT
- R1, R10, R11, R12, R13, R14, R15, R16, R2, R3, R4, R5, R6, R7, R8, R9: value R_Small -> TBD
Connections:
- net VCC renamed +5VD
- net Vdrive renamed +15V
- no-connect marks 6 -> 10
Other:
- moved on the sheet: C1, C10, C11, C12, C13, C2, C3, C4, C5, C6, C7, C8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

Commit message: Minor changes
Parts:
- removed H1, H2, H3, H4: MountingHole_Pad, MountingHole:MountingHole_3.2mm_M3_Pad_Via, symbol Mechanical:MountingHole_Pad
- C1, C10, C11, C2, C7, C8, C9: Manufacturer (none) -> 08055C104KAT2A; RS (none) -> 464-6688
- C12, C13: Manufacturer (none) -> C2012X7R1A106K125AC; Mouser (none) -> 81-GRM21BR71A106KA3K; RS (none) -> 788-3017
- C3, C4, C5, C6: Manufacturer (none) -> EEEFP1E331AP; Mouser (none) -> 667-EEE-HA1E331UP; RS (none) -> 568-525
- D57: value D_TVS -> 6V TVS; Manufacturer (none) -> SMAJ6.0CA-TR; Mouser (none) -> 652-SMAJ6.0CA; RS (none) -> 171-4263
- D58, D59, D60, D61: value 5V -> 5V TVS; Mouser (none) -> 576-AQ05C-01FTG; RS (none) -> 187-1547
- D62: value D_TVS -> 16V TVS; Manufacturer (none) -> SMAJ16CA-E3/61; RS (none) -> 814-1386
- J1: value DC IN -> Conn_02x04_Odd_Even; Mouser (none) -> 855-M20-8890845
- J2: value DC OUT -> Conn_02x04_Odd_Even; Mouser (none) -> 855-M20-7910842R
- J3: value Signal in -> Conn_02x04_Odd_Even; Mouser (none) -> 855-M20-7910842R
- J4: value Signal out -> Conn_02x04_Odd_Even; Mouser (none) -> 855-M20-8890845
- R1, R2: value TBD -> 1k58; Mouser (none) -> 603-RT0805DRE071K58L; RS (none) -> 123-1691
- R10, R11, R12, R13, R14, R15, R16, R3, R4, R5, R6, R7, R8, R9: value TBD -> 0R; Manufacturer (none) -> CRCW08050000Z0EA; RS (none) -> 679-0800
- U1, U2: Mouser (none) -> 595-TLC5952DAP
- U3: Manufacturer (none) -> SN74LS244DW; Mouser (none) -> 595-SN74LS244DWR; RS (none) -> 121-8344
Other:
- moved on the sheet: C10, C11, C4
